Commit message: made updated 'abb_on_axis' URDF

File: setup/catkin/princeton_cell/urdf/_OLD_abb_on_axis.urdf (robot description, URDF)
Before this commit: robot abb_on_axis, 13 links, 12 joints
Links:
- link gripper: geometry collision mesh filename=package://princeton_cell/meshes/collision/gripper.stl; visual mesh filename=package://princeton_cell/meshes/visual/gripper.stl
