Commit message: split up into track, 2rob, 3rob folders

File: setup/catkin/ECL_tracks/urdf/abb_on_axis.urdf (robot description, URDF)
Before this commit: robot abb_on_axis, 13 links, 12 joints
Links:
- link axis: geometry collision mesh filename=package://ECL_tracks/meshes/collision/axis.stl; visual mesh filename=package://ECL_tracks/meshes/visual/axis.stl
- link cart: geometry collision mesh filename=package://ECL_tracks/meshes/collision/cart.stl; visual mesh filename=package://ECL_tracks/meshes/visual/cart.stl
Joints:
- joint joint_1: limit lower=-3.14159 upper=3.14159 effort=100000 velocity=2.618 -> lower=-3.141592653589793 upper=-3.141592653589793 effort=100000 velocity=2.618
- joint joint_2: limit lower=-1.5708 upper=2.61799 effort=100000 velocity=2.618 -> lower=-1.3089969389957472 upper=2.6179938779914944 effort=100000 velocity=2.618; origin xyz=0.175 0 0.495 rpy=0 -0 0  -> xyz=0.175 0 0.495 rpy=0 0 0 
- joint joint_3: limit lower=-3.14159 upper=1.309 effort=100000 velocity=2.618 -> lower=-3.141592653589793 upper=1.3089969389957472 effort=100000 velocity=2.618; origin xyz=0 0 1.095 rpy=0 -0 0  -> xyz=0 0 1.095 rpy=0 0 0 
- joint joint_4: limit lower=-6.98132 upper=6.98132 effort=10000 velocity=6.2832 -> lower=-6.981317007977318 upper=6.981317007977318 effort=10000 velocity=6.2832; origin xyz=0.332 0 0.175 rpy=0 -0 0  -> xyz=0.332 0 0.175 rpy=0 0 0 
- joint joint_5: limit lower=-2.18166 upper=2.0944 effort=100000 velocity=6.2832 -> lower=-2.181661564992912 upper=2.0943951023931953 effort=100000 velocity=6.2832; origin xyz=0.939 0 0 rpy=0 -0 0  -> xyz=0.939 0 0 rpy=0 0 0 
- joint joint_6: axis 0 0 1 -> 1 0 0; limit lower=-6.98132 upper=6.98132 effort=100000 velocity=7.854 -> lower=-6.981317007977318 upper=6.981317007977318 effort=100000 velocity=7.854; origin xyz=0.135 0 0 rpy=0 1.57076 0  -> xyz=0.135 0 0 rpy=0 0 0 
- joint joint_6-tool0: origin xyz=0 0 0 rpy=0 0 0 -> xyz=0 0 0 rpy=0 1.5707963267948966 0

File: setup/catkin/ECL_tracks/urdf/abb_on_axis.xacro (robot description, xacro)
@@ -2,5 +2,5 @@
 <robot name="abb_on_axis" xmlns:xacro="http://wiki.ros.org/xacro">
   <!-- include files -->
-  <xacro:include filename="$(find princeton_cell)/urdf/abb_on_axis_macro.xacro"/>
+  <xacro:include filename="$(find ECL_tracks)/urdf/abb_on_axis_macro.xacro"/>
   <!-- parameter defs -->
   <xacro:abb_on_axis prefix="" />

File: setup/catkin/ECL_tracks/urdf/abb_on_axis_macro.xacro (robot description, xacro)
@@ -5,5 +5,5 @@
     <xacro:include filename="$(find abb_resources)/urdf/common_materials.xacro"/>
     <xacro:include filename="$(find abb_irb4600_40_255)/urdf/abb_irb4600_40_255_macro.xacro"/>
-    <xacro:include filename="$(find princeton_cell)/urdf/linear_axis.xacro"/>
+    <xacro:include filename="$(find ECL_tracks)/urdf/linear_axis.xacro"/>
     <!-- parameter defs -->
     <xacro:linear_axis prefix="${prefix}"/>

File: setup/catkin/ECL_tracks/urdf/linear_axis.xacro (robot description, xacro)
@@ -12,5 +12,5 @@
       <visual>
         <geometry>
-          <mesh filename="package://princeton_cell/meshes/visual/axis.stl"/>
+          <mesh filename="package://ECL_tracks/meshes/visual/axis.stl"/>
         </geometry>
         <xacro:material_abb_white />
@@ -18,5 +18,5 @@
       <collision>
         <geometry>
-          <mesh filename="package://princeton_cell/meshes/collision/axis.stl"/>
+          <mesh filename="package://ECL_tracks/meshes/collision/axis.stl"/>
         </geometry>
       </collision>
@@ -30,5 +30,5 @@
       <visual>
         <geometry>
-          <mesh filename="package://princeton_cell/meshes/visual/cart.stl"/>
+          <mesh filename="package://ECL_tracks/meshes/visual/cart.stl"/>
         </geometry>
         <xacro:material_abb_white />
@@ -36,5 +36,5 @@
       <collision>
         <geometry>
-          <mesh filename="package://princeton_cell/meshes/collision/cart.stl"/>
+          <mesh filename="package://ECL_tracks/meshes/collision/cart.stl"/>
         </geometry>
       </collision>

File: setup/catkin/princeton_3rob_cell/urdf/princeton_3rob_cell.urdf (robot description, URDF)
Before this commit: robot princeton_3rob_cell, 39 links, 38 joints
Links:
- link r1_axis: geometry collision mesh filename=package://ECL_tracks/meshes/collision/axis.stl; visual mesh filename=package://ECL_tracks/meshes/visual/axis.stl
- link r1_cart: geometry collision mesh filename=package://ECL_tracks/meshes/collision/cart.stl; visual mesh filename=package://ECL_tracks/meshes/visual/cart.stl
- link r2_axis: geometry collision mesh filename=package://ECL_tracks/meshes/collision/axis.stl; visual mesh filename=package://ECL_tracks/meshes/visual/axis.stl
- link r2_cart: geometry collision mesh filename=package://ECL_tracks/meshes/collision/cart.stl; visual mesh filename=package://ECL_tracks/meshes/visual/cart.stl
Joints:
- joint r1_joint_1: limit lower=-3.14159 upper=3.14159 effort=100000 velocity=2.618 -> lower=-3.141592653589793 upper=-3.141592653589793 effort=100000 velocity=2.618
- joint r1_joint_2: limit lower=-1.5708 upper=2.61799 effort=100000 velocity=2.618 -> lower=-1.3089969389957472 upper=2.6179938779914944 effort=100000 velocity=2.618; origin xyz=0.175 0 0.495 rpy=0 -0 0  -> xyz=0.175 0 0.495 rpy=0 0 0 
- joint r1_joint_3: limit lower=-3.14159 upper=1.309 effort=100000 velocity=2.618 -> lower=-3.141592653589793 upper=1.3089969389957472 effort=100000 velocity=2.618; origin xyz=0 0 1.095 rpy=0 -0 0  -> xyz=0 0 1.095 rpy=0 0 0 
- joint r1_joint_4: limit lower=-6.98132 upper=6.98132 effort=10000 velocity=6.2832 -> lower=-6.981317007977318 upper=6.981317007977318 effort=10000 velocity=6.2832
- joint r1_joint_5: limit lower=-2.18166 upper=2.0944 effort=100000 velocity=6.2832 -> lower=-2.181661564992912 upper=2.0943951023931953 effort=100000 velocity=6.2832
- joint r1_joint_6: limit lower=-6.98132 upper=6.98132 effort=100000 velocity=7.854 -> lower=-6.981317007977318 upper=6.981317007977318 effort=100000 velocity=7.854
- joint r2_joint_1: limit lower=-3.14159 upper=3.14159 effort=100000 velocity=2.618 -> lower=-3.141592653589793 upper=-3.141592653589793 effort=100000 velocity=2.618
- joint r2_joint_2: limit lower=-1.5708 upper=2.61799 effort=100000 velocity=2.618 -> lower=-1.3089969389957472 upper=2.6179938779914944 effort=100000 velocity=2.618; origin xyz=0.175 0 0.495 rpy=0 -0 0  -> xyz=0.175 0 0.495 rpy=0 0 0 
- joint r2_joint_3: limit lower=-3.14159 upper=1.309 effort=100000 velocity=2.618 -> lower=-3.141592653589793 upper=1.3089969389957472 effort=100000 velocity=2.618; origin xyz=0 0 1.095 rpy=0 -0 0  -> xyz=0 0 1.095 rpy=0 0 0 
- joint r2_joint_4: limit lower=-6.98132 upper=6.98132 effort=10000 velocity=6.2832 -> lower=-6.981317007977318 upper=6.981317007977318 effort=10000 velocity=6.2832
- joint r2_joint_5: limit lower=-2.18166 upper=2.0944 effort=100000 velocity=6.2832 -> lower=-2.181661564992912 upper=2.0943951023931953 effort=100000 velocity=6.2832
- joint r2_joint_6: limit lower=-6.98132 upper=6.98132 effort=100000 velocity=7.854 -> lower=-6.981317007977318 upper=6.981317007977318 effort=100000 velocity=7.854
- joint r3_world_joint: origin xyz=5.3 1.725 -0.3 rpy=0.0 0.0 3.14159 -> xyz=0.0 0.0 0.0 rpy=0.0 0.0 0.0

File: setup/catkin/princeton_3rob_cell/urdf/princeton_3rob_cell.xacro (robot description, xacro)
@@ -1,5 +1,5 @@
 <?xml version="1.0"?>
 <robot name="princeton_3rob_cell" xmlns:xacro="http://wiki.ros.org/xacro">
-  <xacro:include filename="$(find princeton_cell)/urdf/princeton_3rob_cell_macro.xacro"/>
+  <xacro:include filename="$(find princeton_3rob_cell)/urdf/princeton_3rob_cell_macro.xacro"/>
   <xacro:princeton_3rob_cell />
 </robot>

File: setup/catkin/princeton_3rob_cell/urdf/princeton_3rob_cell_macro.xacro (robot description, xacro)
@@ -4,5 +4,5 @@
     <!-- include files -->
     <xacro:include filename="$(find abb_irb7600_400_255)/urdf/abb_irb7600_400_255_macro.xacro"/>
-    <xacro:include filename="$(find princeton_cell)/urdf/abb_on_axis_macro.xacro"/>
+    <xacro:include filename="$(find ECL_tracks)/urdf/abb_on_axis_macro.xacro"/>
     <link name="world" />
     <!-- -->
@@ -11,5 +11,5 @@
       <parent link="world" />
       <child link = "r1_axis" />
-      <origin xyz="3.70 3.45 0.02" rpy="0.0 0.0 3.14159" />
+      <origin rpy="0.0 0.0 3.14159" xyz="3.70 3.45 0.02"/>
     </joint>
     <xacro:abb_on_axis prefix="r1_" />
@@ -27,5 +27,5 @@
       <parent link="world" />
       <child link = "r3_base_link" />
-      <origin xyz="5.3 1.725 -0.3" rpy="0.0 0.0 3.14159" />
+      <origin xyz="0.0 0.0 0.0" rpy="0.0 0.0 0.0" />
     </joint>
     <xacro:abb_irb7600_400_255 prefix="r3_" />

File: setup/catkin/princeton_cell/urdf/princeton_cell.urdf (robot description, URDF)
Before this commit: robot princeton_cell, 27 links, 26 joints
Links:
- link r1_axis: geometry collision mesh filename=package://ECL_tracks/meshes/collision/axis.stl; visual mesh filename=package://ECL_tracks/meshes/visual/axis.stl
- link r1_cart: geometry collision mesh filename=package://ECL_tracks/meshes/collision/cart.stl; visual mesh filename=package://ECL_tracks/meshes/visual/cart.stl
- link r2_axis: geometry collision mesh filename=package://ECL_tracks/meshes/collision/axis.stl; visual mesh filename=package://ECL_tracks/meshes/visual/axis.stl
- link r2_cart: geometry collision mesh filename=package://ECL_tracks/meshes/collision/cart.stl; visual mesh filename=package://ECL_tracks/meshes/visual/cart.stl
Joints:
- joint r1_joint_1: limit lower=-3.14159 upper=3.14159 effort=100000 velocity=2.618 -> lower=-3.141592653589793 upper=-3.141592653589793 effort=100000 velocity=2.618
- joint r1_joint_2: limit lower=-1.5708 upper=2.61799 effort=100000 velocity=2.618 -> lower=-1.3089969389957472 upper=2.6179938779914944 effort=100000 velocity=2.618; origin xyz=0.175 0 0.495 rpy=0 -0 0  -> xyz=0.175 0 0.495 rpy=0 0 0 
- joint r1_joint_3: limit lower=-3.14159 upper=1.309 effort=100000 velocity=2.618 -> lower=-3.141592653589793 upper=1.3089969389957472 effort=100000 velocity=2.618; origin xyz=0 0 1.095 rpy=0 -0 0  -> xyz=0 0 1.095 rpy=0 0 0 
- joint r1_joint_4: limit lower=-6.98132 upper=6.98132 effort=10000 velocity=6.2832 -> lower=-6.981317007977318 upper=6.981317007977318 effort=10000 velocity=6.2832
- joint r1_joint_5: limit lower=-2.18166 upper=2.0944 effort=100000 velocity=6.2832 -> lower=-2.181661564992912 upper=2.0943951023931953 effort=100000 velocity=6.2832
- joint r1_joint_6: limit lower=-6.98132 upper=6.98132 effort=100000 velocity=7.854 -> lower=-6.981317007977318 upper=6.981317007977318 effort=100000 velocity=7.854
- joint r2_joint_1: limit lower=-3.14159 upper=3.14159 effort=100000 velocity=2.618 -> lower=-3.141592653589793 upper=-3.141592653589793 effort=100000 velocity=2.618
- joint r2_joint_2: limit lower=-1.5708 upper=2.61799 effort=100000 velocity=2.618 -> lower=-1.3089969389957472 upper=2.6179938779914944 effort=100000 velocity=2.618; origin xyz=0.175 0 0.495 rpy=0 -0 0  -> xyz=0.175 0 0.495 rpy=0 0 0 
- joint r2_joint_3: limit lower=-3.14159 upper=1.309 effort=100000 velocity=2.618 -> lower=-3.141592653589793 upper=1.3089969389957472 effort=100000 velocity=2.618; origin xyz=0 0 1.095 rpy=0 -0 0  -> xyz=0 0 1.095 rpy=0 0 0 
- joint r2_joint_4: limit lower=-6.98132 upper=6.98132 effort=10000 velocity=6.2832 -> lower=-6.981317007977318 upper=6.981317007977318 effort=10000 velocity=6.2832
- joint r2_joint_5: limit lower=-2.18166 upper=2.0944 effort=100000 velocity=6.2832 -> lower=-2.181661564992912 upper=2.0943951023931953 effort=100000 velocity=6.2832
- joint r2_joint_6: limit lower=-6.98132 upper=6.98132 effort=100000 velocity=7.854 -> lower=-6.981317007977318 upper=6.981317007977318 effort=100000 velocity=7.854

File: setup/catkin/princeton_cell/urdf/princeton_cell_macro.xacro (robot description, xacro)
@@ -3,5 +3,5 @@
   <xacro:macro name="princeton_cell">
     <!-- include files -->
-    <xacro:include filename="$(find princeton_cell)/urdf/abb_on_axis_macro.xacro"/>
+    <xacro:include filename="$(find ECL_tracks)/urdf/abb_on_axis_macro.xacro"/>
     <link name="world" />
     <!-- -->
