Commit message: renamed "ECL_tracks" to "abb_on_axis" sep folder

File: setup/catkin/abb_on_axis/urdf/abb_on_axis.urdf (robot description, URDF)
Before this commit: robot abb_on_axis, 13 links, 12 joints
Links:
- link axis: geometry collision mesh filename=package://abb_on_axis/meshes/collision/axis.stl; visual mesh filename=package://abb_on_axis/meshes/visual/axis.stl
- link cart: geometry collision mesh filename=package://abb_on_axis/meshes/collision/cart.stl; visual mesh filename=package://abb_on_axis/meshes/visual/cart.stl
Joints:
- joint joint_1: limit lower=-3.141592653589793 upper=-3.141592653589793 effort=100000 velocity=2.618 -> lower=-3.141592653589793 upper=3.141592653589793 effort=100000 velocity=2.618

File: setup/catkin/abb_on_axis/urdf/abb_on_axis.xacro (robot description, xacro)
@@ -2,5 +2,5 @@
 <robot name="abb_on_axis" xmlns:xacro="http://wiki.ros.org/xacro">
   <!-- include files -->
-  <xacro:include filename="$(find ECL_tracks)/urdf/abb_on_axis_macro.xacro"/>
+  <xacro:include filename="$(find abb_on_axis)/urdf/abb_on_axis_macro.xacro"/>
   <!-- parameter defs -->
   <xacro:abb_on_axis prefix="" />

File: setup/catkin/abb_on_axis/urdf/abb_on_axis_macro.xacro (robot description, xacro)
@@ -5,5 +5,5 @@
     <xacro:include filename="$(find abb_resources)/urdf/common_materials.xacro"/>
     <xacro:include filename="$(find abb_irb4600_40_255)/urdf/abb_irb4600_40_255_macro.xacro"/>
-    <xacro:include filename="$(find ECL_tracks)/urdf/linear_axis.xacro"/>
+    <xacro:include filename="$(find abb_on_axis)/urdf/linear_axis.xacro"/>
     <!-- parameter defs -->
     <xacro:linear_axis prefix="${prefix}"/>

File: setup/catkin/abb_on_axis/urdf/linear_axis.xacro (robot description, xacro)
@@ -12,5 +12,5 @@
       <visual>
         <geometry>
-          <mesh filename="package://ECL_tracks/meshes/visual/axis.stl"/>
+          <mesh filename="package://abb_on_axis/meshes/visual/axis.stl"/>
         </geometry>
         <xacro:material_abb_white />
@@ -18,5 +18,5 @@
       <collision>
         <geometry>
-          <mesh filename="package://ECL_tracks/meshes/collision/axis.stl"/>
+          <mesh filename="package://abb_on_axis/meshes/collision/axis.stl"/>
         </geometry>
       </collision>
@@ -30,5 +30,5 @@
       <visual>
         <geometry>
-          <mesh filename="package://ECL_tracks/meshes/visual/cart.stl"/>
+          <mesh filename="package://abb_on_axis/meshes/visual/cart.stl"/>
         </geometry>
         <xacro:material_abb_white />
@@ -36,5 +36,5 @@
       <collision>
         <geometry>
-          <mesh filename="package://ECL_tracks/meshes/collision/cart.stl"/>
+          <mesh filename="package://abb_on_axis/meshes/collision/cart.stl"/>
         </geometry>
       </collision>

File: setup/catkin/princeton_3rob_cell/urdf/princeton_3rob_cell.urdf (robot description, URDF)
Before this commit: robot princeton_3rob_cell, 39 links, 38 joints
Links:
- link r1_axis: geometry collision mesh filename=package://abb_on_axis/meshes/collision/axis.stl; visual mesh filename=package://abb_on_axis/meshes/visual/axis.stl
- link r1_cart: geometry collision mesh filename=package://abb_on_axis/meshes/collision/cart.stl; visual mesh filename=package://abb_on_axis/meshes/visual/cart.stl
- link r2_axis: geometry collision mesh filename=package://abb_on_axis/meshes/collision/axis.stl; visual mesh filename=package://abb_on_axis/meshes/visual/axis.stl
- link r2_cart: geometry collision mesh filename=package://abb_on_axis/meshes/collision/cart.stl; visual mesh filename=package://abb_on_axis/meshes/visual/cart.stl

File: setup/catkin/princeton_3rob_cell/urdf/princeton_3rob_cell_macro.xacro (robot description, xacro)
@@ -4,5 +4,5 @@
     <!-- include files -->
     <xacro:include filename="$(find abb_irb7600_400_255)/urdf/abb_irb7600_400_255_macro.xacro"/>
-    <xacro:include filename="$(find ECL_tracks)/urdf/abb_on_axis_macro.xacro"/>
+    <xacro:include filename="$(find abb_on_axis)/urdf/abb_on_axis_macro.xacro"/>
     <link name="world" />
     <!-- -->

File: setup/catkin/princeton_cell/urdf/princeton_cell.urdf (robot description, URDF)
Before this commit: robot princeton_cell, 27 links, 26 joints
Links:
- link r1_axis: geometry collision mesh filename=package://abb_on_axis/meshes/collision/axis.stl; visual mesh filename=package://abb_on_axis/meshes/visual/axis.stl
- link r1_cart: geometry collision mesh filename=package://abb_on_axis/meshes/collision/cart.stl; visual mesh filename=package://abb_on_axis/meshes/visual/cart.stl
- link r2_axis: geometry collision mesh filename=package://abb_on_axis/meshes/collision/axis.stl; visual mesh filename=package://abb_on_axis/meshes/visual/axis.stl
- link r2_cart: geometry collision mesh filename=package://abb_on_axis/meshes/collision/cart.stl; visual mesh filename=package://abb_on_axis/meshes/visual/cart.stl

File: setup/catkin/princeton_cell/urdf/princeton_cell_macro.xacro (robot description, xacro)
@@ -3,5 +3,5 @@
   <xacro:macro name="princeton_cell">
     <!-- include files -->
-    <xacro:include filename="$(find ECL_tracks)/urdf/abb_on_axis_macro.xacro"/>
+    <xacro:include filename="$(find abb_on_axis)/urdf/abb_on_axis_macro.xacro"/>
     <link name="world" />
     <!-- -->
