Commit message: regen .urdf, saved old, mvd gripr out of pton cell

File: setup/catkin/abb_irb4600_40_255/urdf/abb_irb4600_40_255.urdf (robot description, URDF)
Before this commit: robot abb_irb4600_40_255, 9 links, 8 joints
Links:
- added link gripper; collision mesh filename=package://abb_irb4600_40_255/meshes/collision/gripper.stl; visual mesh filename=package://abb_irb4600_40_255/meshes/visual/gripper.stl
- added link tcp
Joints:
- added joint gripper_joint: type fixed, parent tool0, child gripper, origin xyz=0 0 0 rpy=0 0 0
- added joint tcp_joint: type fixed, parent gripper, child tcp, origin xyz=0 0 0.352 rpy=0 0 0

File: setup/catkin/abb_irb4600_40_255/urdf/abb_irb4600_40_255_macro.xacro (robot description, xacro)
@@ -3,4 +3,6 @@
   <xacro:include filename="$(find abb_resources)/urdf/common_materials.xacro"/>
   <xacro:macro name="abb_irb4600_40_255" params="prefix">
+    <xacro:include filename="$(find abb_irb4600_40_255)/urdf/gripper.xacro" />
+    <xacro:gripper prefix="${prefix}" connected_to="${prefix}tool0"/>
     <!-- IRB4600 -->
     <!-- irb4600 link list -->

File: setup/catkin/abb_irb4600_40_255/urdf/gripper.xacro (robot description, xacro)
@@ -7,10 +7,10 @@
       <visual>
         <geometry>
-          <mesh filename="package://princeton_cell/meshes/visual/gripper.stl"/>
+          <mesh filename="package://abb_irb4600_40_255/meshes/visual/gripper.stl"/>
         </geometry>
       </visual>
       <collision>
         <geometry>
-          <mesh filename="package://princeton_cell/meshes/collision/gripper.stl"/>
+          <mesh filename="package://abb_irb4600_40_255/meshes/collision/gripper.stl"/>
         </geometry>
       </collision>

File: setup/catkin/abb_irb7600_400_255/urdf/abb_irb7600_400_255.urdf (robot description, URDF)
Before this commit: robot abb_irb7600_400_255, 12 links, 11 joints
Links:
- link gripper: geometry collision mesh filename=package://abb_irb7600_400_255/meshes/collision/gripper.stl; visual mesh filename=package://abb_irb7600_400_255/meshes/visual/gripper.stl

File: setup/catkin/abb_irb7600_400_255/urdf/abb_irb7600_400_255_macro.xacro (robot description, xacro)
@@ -3,5 +3,5 @@
   <xacro:include filename="$(find abb_resources)/urdf/common_materials.xacro"/>
   <xacro:macro name="abb_irb7600_400_255" params="prefix">
-    <xacro:include filename="$(find princeton_cell)/urdf/gripper.xacro" />
+    <xacro:include filename="$(find abb_irb7600_400_255)/urdf/gripper.xacro" />
     <xacro:gripper prefix="${prefix}" connected_to="${prefix}tool0"/>
     <!-- IRB7600-->

File: setup/catkin/princeton_cell/urdf/_OLD_princeton_cell.urdf (robot description, URDF)
Before this commit: robot princeton_3rob_cell, 39 links, 38 joints
Links:
- removed link r3_balancer_piston
- removed link r3_base
- removed link r3_base_link
- removed link r3_gripper
- removed link r3_link_1
- removed link r3_link_2
- removed link r3_link_3
- removed link r3_link_4
- removed link r3_link_5
- removed link r3_link_6
- removed link r3_tcp
- removed link r3_tool0
Joints:
- removed joint r3_base_link-base
- removed joint r3_gripper_joint
- removed joint r3_joint_1
- removed joint r3_joint_2
- removed joint r3_joint_3
- removed joint r3_joint_4
- removed joint r3_joint_5
- removed joint r3_joint_6
- removed joint r3_joint_6-tool0
- removed joint r3_joint_balancer_piston
- removed joint r3_tcp_joint
- removed joint r3_world_joint

File: setup/catkin/princeton_cell/urdf/abb_on_axis_macro.xacro (robot description, xacro)
@@ -5,10 +5,8 @@
     <xacro:include filename="$(find abb_resources)/urdf/common_materials.xacro"/>
     <xacro:include filename="$(find abb_irb4600_40_255)/urdf/abb_irb4600_40_255_macro.xacro"/>
-    <xacro:include filename="$(find princeton_cell)/urdf/gripper.xacro" />
     <xacro:include filename="$(find princeton_cell)/urdf/linear_axis.xacro"/>
     <!-- parameter defs -->
     <xacro:linear_axis prefix="${prefix}"/>
     <xacro:abb_irb4600_40_255 prefix="${prefix}"/>
-    <xacro:gripper prefix="${prefix}" connected_to="${prefix}tool0"/>
   </xacro:macro>
 </robot>

File: setup/catkin/princeton_cell/urdf/princeton_3rob_cell.urdf (robot description, URDF)
Before this commit: robot princeton_cell, 27 links, 26 joints
Links:
- added link r3_balancer_piston; collision mesh filename=package://abb_irb7600_400_255/meshes/collision/balancer_pis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; visual mesh filename=package://abb_irb7600_400_255/meshes/visual/balancer_piston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
- added link r3_base
- added link r3_base_link; collision mesh filename=package://abb_irb7600_400_255/meshes/collision/base_link.stl; visual mesh filename=package://abb_irb7600_400_255/meshes/visual/base_link.stl
- added link r3_gripper; collision mesh filename=package://abb_irb7600_400_255/meshes/collision/gripper.stl; visual mesh filename=package://abb_irb7600_400_255/meshes/visual/gripper.stl
- added link r3_link_1; collision mesh filename=package://abb_irb7600_400_255/meshes/collision/link_1.stl; visual mesh filename=package://abb_irb7600_400_255/meshes/visual/link_1.stl
- added link r3_link_2; collision mesh filename=package://abb_irb7600_400_255/meshes/collision/link_2.stl; visual mesh filename=package://abb_irb7600_400_255/meshes/visual/link_2.stl
- added link r3_link_3; collision mesh filename=package://abb_irb7600_400_255/meshes/collision/link_3.stl; visual mesh filename=package://abb_irb7600_400_255/meshes/visual/link_3.stl
- added link r3_link_4; collision mesh filename=package://abb_irb7600_support/meshes/irb7600_150_350/collis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; visual mesh filename=package://abb_irb7600_support/meshes/irb7600_150_350/visual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
- added link r3_link_5; collision mesh filename=package://abb_irb7600_400_255/meshes/collision/link_5.stl; visual mesh filename=package://abb_irb7600_400_255/meshes/visual/link_5.stl
- added link r3_link_6; collision mesh filename=package://abb_irb7600_400_255/meshes/collision/link_6.stl; visual mesh filename=package://abb_irb7600_400_255/meshes/visual/link_6.stl
- added link r3_tcp
- added link r3_tool0
- link r1_gripper: geometry collision mesh filename=package://abb_irb4600_40_255/meshes/collision/gripper.stl; visual mesh filename=package://abb_irb4600_40_255/meshes/visual/gripper.stl
- link r2_gripper: geometry collision mesh filename=package://abb_irb4600_40_255/meshes/collision/gripper.stl; visual mesh filename=package://abb_irb4600_40_255/meshes/visual/gripper.stl
Joints:
- added joint r3_base_link-base: type fixed, parent r3_base_link, child r3_base, origin xyz=0 0 0 rpy=0 0 0
- added joint r3_gripper_joint: type fixed, parent r3_tool0, child r3_gripper, origin xyz=0 0 0 rpy=0 0 0
- added joint r3_joint_1: type revolute, parent r3_base_link, child r3_link_1, origin xyz=0 0 0 rpy=0 0 0, axis 0 0 1, limit lower=-3.141592653589793 upper=3.141592653589793 effort=0 velocity=1.7453292519943295
- added joint r3_joint_2: type revolute, parent r3_link_1, child r3_link_2, origin xyz=0.410 0 0.780 rpy=0 0 0, axis 0 1 0, limit lower=-1.0471975511965976 upper=1.4835298641951802 effort=0 velocity=1.0471975511965976
- added joint r3_joint_3: type revolute, parent r3_link_2, child r3_link_3, origin xyz=0 0 1.075 rpy=0 0 0, axis 0 1 0, limit lower=-3.141592653589793 upper=1.0471975511965976 effort=0 velocity=1.0471975511965976
- added joint r3_joint_4: type revolute, parent r3_link_3, child r3_link_4, origin xyz=0 0 0.165 rpy=0 0 0, axis 1 0 0, limit lower=-5.235987755982989 upper=5.235987755982989 effort=0 velocity=1.7453292519943295
- added joint r3_joint_5: type revolute, parent r3_link_4, child r3_link_5, origin xyz=2.012 0 0 rpy=0 0 0, axis 0 1 0, limit lower=-1.7453292519943295 upper=1.7453292519943295 effort=0 velocity=1.7453292519943295
- added joint r3_joint_6: type revolute, parent r3_link_5, child r3_link_6, origin xyz=0.250 0 0 rpy=0 0 0, axis 1 0 0, limit lower=-6.283185307179586 upper=6.283185307179586 effort=0 velocity=3.3161255787892263
- added joint r3_joint_6-tool0: type fixed, parent r3_link_6, child r3_tool0, origin xyz=0 0 0 rpy=0 1.5707963267948966 0
- added joint r3_joint_balancer_piston: type fixed, parent r3_link_1, child r3_balancer_piston, origin xyz=-0.380 0 0.6545 rpy=0 0 0
- added joint r3_tcp_joint: type fixed, parent r3_gripper, child r3_tcp, origin xyz=0 0 0.352 rpy=0 0 0
- added joint r3_world_joint: type fixed, parent world, child r3_base_link, origin xyz=0.0 0.0 0.0 rpy=0.0 0.0 0.0

File: setup/catkin/princeton_cell/urdf/princeton_cell.urdf (robot description, URDF)
Before this commit: robot princeton_cell, 27 links, 26 joints
Links:
- link r1_gripper: geometry collision mesh filename=package://abb_irb4600_40_255/meshes/collision/gripper.stl; visual mesh filename=package://abb_irb4600_40_255/meshes/visual/gripper.stl
- link r2_gripper: geometry collision mesh filename=package://abb_irb4600_40_255/meshes/collision/gripper.stl; visual mesh filename=package://abb_irb4600_40_255/meshes/visual/gripper.stl

Commit message: regenerated all urdfs

File: setup/catkin/abb_irb4600_40_255/urdf/abb_irb4600_40_255.urdf (robot description, URDF)
Before this commit: robot abb_irb4600_40_255, 11 links, 10 joints
Joints:
- joint joint_4: origin xyz=0.332 0 0.175 rpy=0 -0 0  -> xyz=0.332 0 0.175 rpy=0 0 0 
- joint joint_5: origin xyz=0.939 0 0 rpy=0 -0 0  -> xyz=0.939 0 0 rpy=0 0 0 
- joint joint_6: axis 0 0 1 -> 1 0 0; origin xyz=0.135 0 0 rpy=0 1.57076 0  -> xyz=0.135 0 0 rpy=0 0 0 
- joint joint_6-tool0: origin xyz=0 0 0 rpy=0 0 0 -> xyz=0 0 0 rpy=0 1.5707963267948966 0

File: setup/catkin/abb_irb7600_400_255/urdf/abb_irb7600_400_255.urdf (robot description, URDF)
Before this commit: robot abb_irb7600_400_255, 12 links, 11 joints
Joints:
- joint joint_2: origin xyz=0.0 0 0.0 rpy=0 0 0 -> xyz=0.410 0 0.780 rpy=0 0 0
- joint joint_3: origin xyz=0 0 0 rpy=0 0 0 -> xyz=0 0 1.075 rpy=0 0 0
- joint joint_4: origin xyz=0 0 0.0 rpy=0 0 0 -> xyz=0.175 0 0 rpy=0 0 0
- joint joint_5: origin xyz=0 0 0 rpy=0 0 0 -> xyz=0.882 0 0 rpy=0 0 0
- joint joint_6: origin xyz=0 0 0 rpy=0 0 0 -> xyz=0.244 0 0 rpy=0 0 0
- joint joint_6-tool0: origin xyz=1.71 0 2.02 rpy=0 1.5707963267948966 0 -> xyz=0 0 0 rpy=0 1.5707963267948966 0
- joint joint_balancer_piston: origin xyz=0 0 0 rpy=0 0 0 -> xyz=-0.378 0 0.654 rpy=0 0 0

File: setup/catkin/abb_irb7600_400_255/urdf/abb_irb7600_400_255_macro.xacro (robot description, xacro)
@@ -146,5 +146,5 @@
       <parent link="${prefix}link_3"/>
       <child link="${prefix}link_4"/>
-      <origin xyz="0.175 0 0.165" rpy="0 0 0"/>
+      <origin xyz="0.175 0 0" rpy="0 0 0"/>
       <axis xyz="1 0 0"/>
       <limit lower="-${radians(300)}" upper="${radians(300)}" effort="0" velocity="${radians(100)}"/>

File: setup/catkin/princeton_cell/urdf/princeton_3rob_cell.urdf (robot description, URDF)
Before this commit: robot princeton_3rob_cell, 39 links, 38 joints
Joints:
- joint r1_joint_4: origin xyz=0.332 0 0.175 rpy=0 -0 0  -> xyz=0.332 0 0.175 rpy=0 0 0 
- joint r1_joint_5: origin xyz=0.939 0 0 rpy=0 -0 0  -> xyz=0.939 0 0 rpy=0 0 0 
- joint r1_joint_6: axis 0 0 1 -> 1 0 0; origin xyz=0.135 0 0 rpy=0 1.57076 0  -> xyz=0.135 0 0 rpy=0 0 0 
- joint r1_joint_6-tool0: origin xyz=0 0 0 rpy=0 0 0 -> xyz=0 0 0 rpy=0 1.5707963267948966 0
- joint r2_joint_4: origin xyz=0.332 0 0.175 rpy=0 -0 0  -> xyz=0.332 0 0.175 rpy=0 0 0 
- joint r2_joint_5: origin xyz=0.939 0 0 rpy=0 -0 0  -> xyz=0.939 0 0 rpy=0 0 0 
- joint r2_joint_6: axis 0 0 1 -> 1 0 0; origin xyz=0.135 0 0 rpy=0 1.57076 0  -> xyz=0.135 0 0 rpy=0 0 0 
- joint r2_joint_6-tool0: origin xyz=0 0 0 rpy=0 0 0 -> xyz=0 0 0 rpy=0 1.5707963267948966 0
- joint r3_joint_2: origin xyz=0.0 0 0.0 rpy=0 0 0 -> xyz=0.410 0 0.780 rpy=0 0 0
- joint r3_joint_3: origin xyz=0 0 0 rpy=0 0 0 -> xyz=0 0 1.075 rpy=0 0 0
- joint r3_joint_4: origin xyz=0 0 0.0 rpy=0 0 0 -> xyz=0.175 0 0 rpy=0 0 0
- joint r3_joint_5: origin xyz=0 0 0 rpy=0 0 0 -> xyz=0.882 0 0 rpy=0 0 0
- joint r3_joint_6: origin xyz=0 0 0 rpy=0 0 0 -> xyz=0.244 0 0 rpy=0 0 0
- joint r3_joint_6-tool0: origin xyz=1.71 0 2.02 rpy=0 1.5707963267948966 0 -> xyz=0 0 0 rpy=0 1.5707963267948966 0
- joint r3_joint_balancer_piston: origin xyz=0 0 0 rpy=0 0 0 -> xyz=-0.378 0 0.654 rpy=0 0 0

File: setup/catkin/princeton_cell/urdf/princeton_cell.urdf (robot description, URDF)
Before this commit: robot princeton_cell, 27 links, 26 joints
Joints:
- joint r1_joint_4: origin xyz=0.332 0 0.175 rpy=0 -0 0  -> xyz=0.332 0 0.175 rpy=0 0 0 
- joint r1_joint_5: origin xyz=0.939 0 0 rpy=0 -0 0  -> xyz=0.939 0 0 rpy=0 0 0 
- joint r1_joint_6: axis 0 0 1 -> 1 0 0; origin xyz=0.135 0 0 rpy=0 1.57076 0  -> xyz=0.135 0 0 rpy=0 0 0 
- joint r1_joint_6-tool0: origin xyz=0 0 0 rpy=0 0 0 -> xyz=0 0 0 rpy=0 1.5707963267948966 0
- joint r2_joint_4: origin xyz=0.332 0 0.175 rpy=0 -0 0  -> xyz=0.332 0 0.175 rpy=0 0 0 
- joint r2_joint_5: origin xyz=0.939 0 0 rpy=0 -0 0  -> xyz=0.939 0 0 rpy=0 0 0 
- joint r2_joint_6: axis 0 0 1 -> 1 0 0; origin xyz=0.135 0 0 rpy=0 1.57076 0  -> xyz=0.135 0 0 rpy=0 0 0 
- joint r2_joint_6-tool0: origin xyz=0 0 0 rpy=0 0 0 -> xyz=0 0 0 rpy=0 1.5707963267948966 0

Commit message: fixed minus in joint1 of 4600, added 7600 origin

File: setup/catkin/abb_irb4600_40_255/urdf/abb_irb4600_40_255.urdf (robot description, URDF)
Before this commit: robot abb_irb4600_40_255, 11 links, 10 joints
Joints:
- joint joint_1: limit lower=-3.14159 upper=3.14159 effort=100000 velocity=2.618 -> lower=-3.141592653589793 upper=3.141592653589793 effort=100000 velocity=2.618
- joint joint_2: limit lower=-1.5708 upper=2.61799 effort=100000 velocity=2.618 -> lower=-1.3089969389957472 upper=2.6179938779914944 effort=100000 velocity=2.618; origin xyz=0.175 0 0.495 rpy=0 -0 0  -> xyz=0.175 0 0.495 rpy=0 0 0 
- joint joint_3: limit lower=-3.14159 upper=1.309 effort=100000 velocity=2.618 -> lower=-3.141592653589793 upper=1.3089969389957472 effort=100000 velocity=2.618; origin xyz=0 0 1.095 rpy=0 -0 0  -> xyz=0 0 1.095 rpy=0 0 0 
- joint joint_4: limit lower=-6.98132 upper=6.98132 effort=10000 velocity=6.2832 -> lower=-6.981317007977318 upper=6.981317007977318 effort=10000 velocity=6.2832
- joint joint_5: limit lower=-2.18166 upper=2.0944 effort=100000 velocity=6.2832 -> lower=-2.181661564992912 upper=2.0943951023931953 effort=100000 velocity=6.2832
- joint joint_6: limit lower=-6.98132 upper=6.98132 effort=100000 velocity=7.854 -> lower=-6.981317007977318 upper=6.981317007977318 effort=100000 velocity=7.854

File: setup/catkin/abb_irb4600_40_255/urdf/abb_irb4600_40_255_macro.xacro (robot description, xacro)
@@ -140,5 +140,5 @@
       <origin xyz="0 0 0" rpy="0 0 0 "/>
       <axis   xyz="0 0 1"/>
-      <limit lower="-${radians(180)}" upper="-${radians(180)}" effort="100000" velocity="2.618" />
+      <limit lower="-${radians(180)}" upper="${radians(180)}" effort="100000" velocity="2.618" />
       <dynamics damping="0.2" friction="0" />
     </joint>

File: setup/catkin/princeton_3rob_cell/urdf/princeton_3rob_cell.urdf (robot description, URDF)
Before this commit: robot princeton_3rob_cell, 39 links, 38 joints
Joints:
- joint r1_joint_1: limit lower=-3.141592653589793 upper=-3.141592653589793 effort=100000 velocity=2.618 -> lower=-3.141592653589793 upper=3.141592653589793 effort=100000 velocity=2.618
- joint r2_joint_1: limit lower=-3.141592653589793 upper=-3.141592653589793 effort=100000 velocity=2.618 -> lower=-3.141592653589793 upper=3.141592653589793 effort=100000 velocity=2.618
- joint r3_world_joint: origin xyz=0.0 0.0 0.0 rpy=0.0 0.0 0.0 -> xyz=5.3 1.725 -0.3 rpy=0.0 0.0 3.14159

File: setup/catkin/princeton_3rob_cell/urdf/princeton_3rob_cell_macro.xacro (robot description, xacro)
@@ -27,5 +27,5 @@
       <parent link="world" />
       <child link = "r3_base_link" />
-      <origin xyz="0.0 0.0 0.0" rpy="0.0 0.0 0.0" />
+      <origin xyz="5.3 1.725 -0.3" rpy="0.0 0.0 3.14159"/>
     </joint>
     <xacro:abb_irb7600_400_255 prefix="r3_" />

File: setup/catkin/princeton_cell/urdf/princeton_cell.urdf (robot description, URDF)
Before this commit: robot princeton_cell, 27 links, 26 joints
Joints:
- joint r1_joint_1: limit lower=-3.141592653589793 upper=-3.141592653589793 effort=100000 velocity=2.618 -> lower=-3.141592653589793 upper=3.141592653589793 effort=100000 velocity=2.618
- joint r2_joint_1: limit lower=-3.141592653589793 upper=-3.141592653589793 effort=100000 velocity=2.618 -> lower=-3.141592653589793 upper=3.141592653589793 effort=100000 velocity=2.618

Commit message: updat to 4600 mesh and xacro, based on eth

File: setup/catkin/abb_irb4600_40_255/urdf/abb_irb4600_40_255.urdf (robot description, URDF)
Before this commit: robot abb_irb4600_40_255, 11 links, 10 joints
Joints:
- joint joint_1: origin xyz=0 0 0 rpy=0 0 0  -> xyz=0 0 0.495 rpy=0 0 0
- joint joint_2: origin xyz=0.175 0 0.495 rpy=0 0 0  -> xyz=0.175 0 0 rpy=0 0 0
- joint joint_3: origin xyz=0 0 1.095 rpy=0 0 0  -> xyz=0 0 1.095 rpy=0 0 0
- joint joint_4: origin xyz=0.332 0 0.175 rpy=0 0 0  -> xyz=0 0 0.175 rpy=0 0 0
- joint joint_5: origin xyz=0.939 0 0 rpy=0 0 0  -> xyz=1.270 0 0 rpy=0 0 0
- joint joint_6: origin xyz=0.135 0 0 rpy=0 0 0  -> xyz=0.135 0 0 rpy=0 0 0

File: setup/catkin/abb_irb4600_40_255/urdf/abb_irb4600_40_255_macro.xacro (robot description, xacro)
@@ -17,5 +17,5 @@
           <mesh filename="package://abb_irb4600_40_255/meshes/visual/base_link.stl"/>
         </geometry>
-        <xacro:material_abb_graphite_white />
+        <xacro:material_abb_white/>
       </visual>
       <collision>
@@ -23,4 +23,5 @@
           <mesh filename="package://abb_irb4600_40_255/meshes/collision/base_link.stl"/>
         </geometry>
+        <xacro:material_abb_white/>
       </collision>
     </link>
@@ -138,5 +139,5 @@
       <parent link="${prefix}base_link"/>
       <child  link="${prefix}link_1"/>
-      <origin xyz="0 0 0" rpy="0 0 0 "/>
+      <origin xyz="0 0 0.495" rpy="0 0 0"/>
       <axis   xyz="0 0 1"/>
       <limit lower="-${radians(180)}" upper="${radians(180)}" effort="100000" velocity="2.618" />
@@ -146,5 +147,5 @@
       <parent link="${prefix}link_1"/>
       <child  link="${prefix}link_2"/>
-      <origin xyz="0.175 0 0.495" rpy="0 0 0 "/>
+      <origin xyz="0.175 0 0" rpy="0 0 0"/>
       <axis   xyz="0 1 0"/>
       <limit lower="-${radians(75)}" upper="${radians(150)}" effort="100000" velocity="2.618" />
@@ -154,5 +155,5 @@
       <parent link="${prefix}link_2"/>
       <child  link="${prefix}link_3"/>
-      <origin xyz="0 0 1.095" rpy="0 0 0 "/>
+      <origin xyz="0 0 1.095" rpy="0 0 0"/>
       <axis   xyz="0 1 0"/>
       <limit lower="-${radians(180)}" upper="${radians(75)}" effort="100000" velocity="2.618" />
@@ -162,5 +163,5 @@
       <parent link="${prefix}link_3"/>
       <child  link="${prefix}link_4"/>
-      <origin xyz="0.332 0 0.175" rpy="0 0 0 "/>
+      <origin xyz="0 0 0.175" rpy="0 0 0"/>
       <axis   xyz="1 0 0"/>
       <limit lower="-${radians(400)}" upper="${radians(400)}" effort="10000" velocity="6.2832" />
@@ -170,5 +171,5 @@
       <parent link="${prefix}link_4"/>
       <child  link="${prefix}link_5"/>
-      <origin xyz="0.939 0 0" rpy="0 0 0 "/>
+      <origin xyz="1.270 0 0" rpy="0 0 0"/>
       <axis   xyz="0 1 0"/>
       <limit lower="-${radians(125)}" upper="${radians(120)}" effort="100000" velocity="6.2832" />
@@ -178,5 +179,5 @@
       <parent link="${prefix}link_5"/>
       <child  link="${prefix}link_6"/>
-      <origin xyz="0.135 0 0" rpy="0 0 0 "/>
+      <origin xyz="0.135 0 0" rpy="0 0 0"/>
       <axis   xyz="1 0 0"/>
       <limit lower="-${radians(400)}" upper="${radians(400)}" effort="100000" velocity="7.854" />

File: setup/catkin/abb_on_axis/urdf/abb_on_axis.urdf (robot description, URDF)
Before this commit: robot abb_on_axis, 13 links, 12 joints
Joints:
- joint joint_1: origin xyz=0 0 0 rpy=0 0 0  -> xyz=0 0 0.495 rpy=0 0 0
- joint joint_2: origin xyz=0.175 0 0.495 rpy=0 0 0  -> xyz=0.175 0 0 rpy=0 0 0
- joint joint_3: origin xyz=0 0 1.095 rpy=0 0 0  -> xyz=0 0 1.095 rpy=0 0 0
- joint joint_4: origin xyz=0.332 0 0.175 rpy=0 0 0  -> xyz=0 0 0.175 rpy=0 0 0
- joint joint_5: origin xyz=0.939 0 0 rpy=0 0 0  -> xyz=1.270 0 0 rpy=0 0 0
- joint joint_6: origin xyz=0.135 0 0 rpy=0 0 0  -> xyz=0.135 0 0 rpy=0 0 0

File: setup/catkin/princeton_3rob_cell/urdf/princeton_3rob_cell.urdf (robot description, URDF)
Before this commit: robot princeton_3rob_cell, 39 links, 38 joints
Joints:
- joint r1_joint_1: origin xyz=0 0 0 rpy=0 0 0  -> xyz=0 0 0.495 rpy=0 0 0
- joint r1_joint_2: origin xyz=0.175 0 0.495 rpy=0 0 0  -> xyz=0.175 0 0 rpy=0 0 0
- joint r1_joint_3: origin xyz=0 0 1.095 rpy=0 0 0  -> xyz=0 0 1.095 rpy=0 0 0
- joint r1_joint_4: origin xyz=0.332 0 0.175 rpy=0 0 0  -> xyz=0 0 0.175 rpy=0 0 0
- joint r1_joint_5: origin xyz=0.939 0 0 rpy=0 0 0  -> xyz=1.270 0 0 rpy=0 0 0
- joint r1_joint_6: origin xyz=0.135 0 0 rpy=0 0 0  -> xyz=0.135 0 0 rpy=0 0 0
- joint r2_joint_1: origin xyz=0 0 0 rpy=0 0 0  -> xyz=0 0 0.495 rpy=0 0 0
- joint r2_joint_2: origin xyz=0.175 0 0.495 rpy=0 0 0  -> xyz=0.175 0 0 rpy=0 0 0
- joint r2_joint_3: origin xyz=0 0 1.095 rpy=0 0 0  -> xyz=0 0 1.095 rpy=0 0 0
- joint r2_joint_4: origin xyz=0.332 0 0.175 rpy=0 0 0  -> xyz=0 0 0.175 rpy=0 0 0
- joint r2_joint_5: origin xyz=0.939 0 0 rpy=0 0 0  -> xyz=1.270 0 0 rpy=0 0 0
- joint r2_joint_6: origin xyz=0.135 0 0 rpy=0 0 0  -> xyz=0.135 0 0 rpy=0 0 0

File: setup/catkin/princeton_cell/urdf/princeton_cell.urdf (robot description, URDF)
Before this commit: robot princeton_cell, 27 links, 26 joints
Joints:
- joint r1_joint_1: origin xyz=0 0 0 rpy=0 0 0  -> xyz=0 0 0.495 rpy=0 0 0
- joint r1_joint_2: origin xyz=0.175 0 0.495 rpy=0 0 0  -> xyz=0.175 0 0 rpy=0 0 0
- joint r1_joint_3: origin xyz=0 0 1.095 rpy=0 0 0  -> xyz=0 0 1.095 rpy=0 0 0
- joint r1_joint_4: origin xyz=0.332 0 0.175 rpy=0 0 0  -> xyz=0 0 0.175 rpy=0 0 0
- joint r1_joint_5: origin xyz=0.939 0 0 rpy=0 0 0  -> xyz=1.270 0 0 rpy=0 0 0
- joint r1_joint_6: origin xyz=0.135 0 0 rpy=0 0 0  -> xyz=0.135 0 0 rpy=0 0 0
- joint r2_joint_1: origin xyz=0 0 0 rpy=0 0 0  -> xyz=0 0 0.495 rpy=0 0 0
- joint r2_joint_2: origin xyz=0.175 0 0.495 rpy=0 0 0  -> xyz=0.175 0 0 rpy=0 0 0
- joint r2_joint_3: origin xyz=0 0 1.095 rpy=0 0 0  -> xyz=0 0 1.095 rpy=0 0 0
- joint r2_joint_4: origin xyz=0.332 0 0.175 rpy=0 0 0  -> xyz=0 0 0.175 rpy=0 0 0
- joint r2_joint_5: origin xyz=0.939 0 0 rpy=0 0 0  -> xyz=1.270 0 0 rpy=0 0 0
- joint r2_joint_6: origin xyz=0.135 0 0 rpy=0 0 0  -> xyz=0.135 0 0 rpy=0 0 0
