Commit message: some reorg of IRB4600 xacro files (to make clear)

File: setup/catkin/abb_irb4600_40_255/urdf/abb_irb4600_40_255_macro.xacro (robot description, xacro)
@@ -129,5 +129,6 @@
         </geometry>
       </collision>
-    </link>
+    </link>'
+    '
     <link name="${prefix}tool0"/>
     <!-- end of link list -->

File: setup/catkin/princeton_cell/urdf/abb_on_axis_macro.xacro (robot description, xacro)
@@ -7,4 +7,5 @@
     <xacro:include filename="$(find princeton_cell)/urdf/gripper.xacro" />
     <xacro:linear_axis prefix="${prefix}"/>
+    <!-- joint list -->
     <joint name="${prefix}abb_joint" type="fixed">
       <parent link="${prefix}cart"/>
@@ -13,4 +14,5 @@
       <dynamics damping="0.2" friction="0" />
     </joint>
+    <!-- end of joint list -->
     <xacro:abb_irb4600_40_255 prefix="${prefix}"/>
     <xacro:gripper prefix="${prefix}" connected_to="${prefix}tool0"/>

File: setup/catkin/princeton_cell/urdf/gripper.xacro (robot description, xacro)
@@ -3,4 +3,20 @@
   <!-- Here we define the 2 parameters of the macro -->
   <xacro:macro name="gripper" params="prefix connected_to">
+    <!-- link list -->
+    <link name="${prefix}gripper">
+      <visual>
+        <geometry>
+          <mesh filename="package://princeton_cell/meshes/visual/gripper.stl"/>
+        </geometry>
+      </visual>
+      <collision>
+        <geometry>
+          <mesh filename="package://princeton_cell/meshes/collision/gripper.stl"/>
+        </geometry>
+      </collision>
+    </link>
+    <link name="${prefix}tcp"/>
+    <!-- end of link list -->
+    <!-- joint list -->
     <!-- Create a fixed joint with a parameterized name. -->
     <joint name="${prefix}gripper_joint" type="fixed">
@@ -11,18 +27,4 @@
       <origin rpy="0 0 0" xyz="0 0 0"/>
     </joint>
-    <link name="${prefix}gripper">
-      <visual>
-        <geometry>
-          <!-- The path to the visual meshes in the package. -->
-          <mesh filename="package://princeton_cell/meshes/visual/gripper.stl"/>
-        </geometry>
-      </visual>
-      <collision>
-        <geometry>
-          <!-- The path to the collision meshes in the package. -->
-          <mesh filename="package://princeton_cell/meshes/collision/gripper.stl"/>
-        </geometry>
-      </collision>
-    </link>
     <!-- TCP frame -->
     <joint name="${prefix}tcp_joint" type="fixed">
@@ -31,5 +33,5 @@
       <child link="${prefix}tcp"/>
     </joint>
-    <link name="${prefix}tcp"/>
+    <!-- end of joint list -->
   </xacro:macro>
 </robot>

File: setup/catkin/princeton_cell/urdf/linear_axis.xacro (robot description, xacro)
@@ -2,4 +2,5 @@
 <robot xmlns:xacro="http://wiki.ros.org/xacro">
   <xacro:macro name="linear_axis" params="prefix">
+    <!-- link list -->
     <link name="${prefix}axis">
       <inertial>
@@ -20,12 +21,4 @@
       </collision>
     </link>
-    <joint name="${prefix}cart_joint" type="prismatic">
-      <parent link="${prefix}axis"/>
-      <child  link="${prefix}cart"/>
-      <origin xyz="0 0 0" rpy="0 0 0 "/>
-      <axis   xyz="1 0 0"/>
-      <limit lower="0" upper="3.9" effort="100000" velocity="2.618" />
-      <dynamics damping="0.2" friction="0" />
-    </joint>
     <link name="${prefix}cart">
       <inertial>
@@ -46,4 +39,15 @@
       </collision>
     </link>
+    <!-- end of link list -->
+    <!-- joint list -->
+    <joint name="${prefix}cart_joint" type="prismatic">
+      <parent link="${prefix}axis"/>
+      <child  link="${prefix}cart"/>
+      <origin xyz="0 0 0" rpy="0 0 0 "/>
+      <axis   xyz="1 0 0"/>
+      <limit lower="0" upper="3.9" effort="100000" velocity="2.618" />
+      <dynamics damping="0.2" friction="0" />
+    </joint>
+    <!-- end of joint list -->
   </xacro:macro>
 </robot>

Commit message: added some notes to .xacro files for 4600 and 7600

File: setup/catkin/abb_irb4600_40_255/urdf/abb_irb4600_40_255_macro.xacro (robot description, xacro)
@@ -129,6 +129,5 @@
         </geometry>
       </collision>
-    </link>'
-    '
+    </link>
     <link name="${prefix}tool0"/>
     <!-- end of link list -->

File: setup/catkin/abb_irb7600_400_255/urdf/abb_irb7600_400_255.xacro (robot description, xacro)
@@ -2,4 +2,4 @@
 <robot name="abb_irb7600_400_255" xmlns:xacro="http://wiki.ros.org/xacro">
   <xacro:include filename="$(find abb_irb7600_400_255)/urdf/abb_irb7600_400_255_macro.xacro"/>
-  <xacro:abb_irb4600_40_255 prefix=""/>
+  <xacro:abb_irb7600_400_255 prefix=""/>
 </robot>

File: setup/catkin/princeton_cell/urdf/abb_on_axis.xacro (robot description, xacro)
@@ -1,5 +1,9 @@
 <?xml version="1.0"?>
 <robot name="abb_on_axis" xmlns:xacro="http://wiki.ros.org/xacro">
+  <!-- include files -->
   <xacro:include filename="$(find princeton_cell)/urdf/abb_on_axis_macro.xacro"/>
+  <!-- end of include files -->
+  <!-- parameter defs -->
   <xacro:abb_on_axis prefix="" />
+  <!-- end of parameter defs -->
 </robot>

File: setup/catkin/princeton_cell/urdf/abb_on_axis_macro.xacro (robot description, xacro)
@@ -2,9 +2,15 @@
 <robot xmlns:xacro="http://wiki.ros.org/xacro">
   <xacro:macro name="abb_on_axis" params="prefix">
+    <!-- include files -->
     <xacro:include filename="$(find abb_resources)/urdf/common_materials.xacro"/>
     <xacro:include filename="$(find abb_irb4600_40_255)/urdf/abb_irb4600_40_255_macro.xacro"/>
     <xacro:include filename="$(find princeton_cell)/urdf/linear_axis.xacro"/>
     <xacro:include filename="$(find princeton_cell)/urdf/gripper.xacro" />
+    <!-- end of include files -->
+    <!-- parameter defs -->
     <xacro:linear_axis prefix="${prefix}"/>
+    <xacro:abb_irb4600_40_255 prefix="${prefix}"/>
+    <xacro:gripper prefix="${prefix}" connected_to="${prefix}tool0"/>
+    <!-- end of parameter defs -->
     <!-- joint list -->
     <joint name="${prefix}abb_joint" type="fixed">
@@ -15,6 +21,4 @@
     </joint>
     <!-- end of joint list -->
-    <xacro:abb_irb4600_40_255 prefix="${prefix}"/>
-    <xacro:gripper prefix="${prefix}" connected_to="${prefix}tool0"/>
   </xacro:macro>
 </robot>

File: setup/catkin/princeton_cell/urdf/princeton_cell_macro.xacro (robot description, xacro)
@@ -2,5 +2,7 @@
 <robot xmlns:xacro="http://wiki.ros.org/xacro">
   <xacro:macro name="princeton_cell">
+    <!-- include files -->
     <xacro:include filename="$(find princeton_cell)/urdf/abb_on_axis_macro.xacro"/>
+    <!-- end include files -->
     <link name="world" />
     <joint name="r2_world_joint" type="fixed">

Commit message: add stls for IRB7600, clean xacros for pton cell

File: setup/catkin/abb_irb4600_40_255/urdf/abb_irb4600_40_255_macro.xacro (robot description, xacro)
@@ -3,5 +3,6 @@
   <xacro:include filename="$(find abb_resources)/urdf/common_materials.xacro"/>
   <xacro:macro name="abb_irb4600_40_255" params="prefix">
-    <!-- link list -->
+    <!-- IRB4600 -->
+    <!-- irb4600 link list -->
     <link name="${prefix}base_link">
       <inertial>
@@ -131,6 +132,5 @@
     </link>
     <link name="${prefix}tool0"/>
-    <!-- end of link list -->
-    <!-- joint list -->
+    <!-- irb4600 joint list -->
     <joint name="${prefix}joint_1" type="revolute">
       <parent link="${prefix}base_link"/>
@@ -186,6 +186,6 @@
       <origin xyz="0 0 0" rpy="0 0 0"/>
     </joint>
-    <!-- end of joint list -->
-    <!-- ROS base_link to ABB World Coordinates transform -->
+    <!-- -->
+    <!-- IRB4600 base_link to ABB World Coordinates transform -->
     <link name="${prefix}base" />
     <joint name="${prefix}base_link-base" type="fixed">

File: setup/catkin/princeton_cell/urdf/abb_on_axis.xacro (robot description, xacro)
@@ -3,7 +3,5 @@
   <!-- include files -->
   <xacro:include filename="$(find princeton_cell)/urdf/abb_on_axis_macro.xacro"/>
-  <!-- end of include files -->
   <!-- parameter defs -->
   <xacro:abb_on_axis prefix="" />
-  <!-- end of parameter defs -->
 </robot>

File: setup/catkin/princeton_cell/urdf/abb_on_axis_macro.xacro (robot description, xacro)
@@ -5,20 +5,10 @@
     <xacro:include filename="$(find abb_resources)/urdf/common_materials.xacro"/>
     <xacro:include filename="$(find abb_irb4600_40_255)/urdf/abb_irb4600_40_255_macro.xacro"/>
+    <xacro:include filename="$(find princeton_cell)/urdf/gripper.xacro" />
     <xacro:include filename="$(find princeton_cell)/urdf/linear_axis.xacro"/>
-    <xacro:include filename="$(find princeton_cell)/urdf/gripper.xacro" />
-    <!-- end of include files -->
     <!-- parameter defs -->
     <xacro:linear_axis prefix="${prefix}"/>
     <xacro:abb_irb4600_40_255 prefix="${prefix}"/>
     <xacro:gripper prefix="${prefix}" connected_to="${prefix}tool0"/>
-    <!-- end of parameter defs -->
-    <!-- joint list -->
-    <joint name="${prefix}abb_joint" type="fixed">
-      <parent link="${prefix}cart"/>
-      <child  link="${prefix}base_link"/>
-      <origin xyz="0 0 0 " rpy="0 0 ${pi/2} "/>
-      <dynamics damping="0.2" friction="0" />
-    </joint>
-    <!-- end of joint list -->
   </xacro:macro>
 </robot>

File: setup/catkin/princeton_cell/urdf/gripper.xacro (robot description, xacro)
@@ -1,7 +1,7 @@
 <?xml version="1.0" encoding="utf-8"?>
 <robot xmlns:xacro="https://ros.org/wiki/xacro">
-  <!-- Here we define the 2 parameters of the macro -->
   <xacro:macro name="gripper" params="prefix connected_to">
-    <!-- link list -->
+    <!-- GRIPPER -->
+    <!-- gripper link list -->
     <link name="${prefix}gripper">
       <visual>
@@ -17,15 +17,10 @@
     </link>
     <link name="${prefix}tcp"/>
-    <!-- end of link list -->
-    <!-- joint list -->
-    <!-- Create a fixed joint with a parameterized name. -->
+    <!-- gripper joint list -->
     <joint name="${prefix}gripper_joint" type="fixed">
-      <!-- The parent link must be read from the robot model it is attached to. -->
       <parent link="${connected_to}"/>
       <child link="${prefix}gripper"/>
-      <!-- The tool is directly attached to the flange. -->
       <origin rpy="0 0 0" xyz="0 0 0"/>
     </joint>
-    <!-- TCP frame -->
     <joint name="${prefix}tcp_joint" type="fixed">
       <origin xyz="0 0 0.352" rpy="0 0 0"/>
@@ -33,5 +28,4 @@
       <child link="${prefix}tcp"/>
     </joint>
-    <!-- end of joint list -->
   </xacro:macro>
 </robot>

File: setup/catkin/princeton_cell/urdf/linear_axis.xacro (robot description, xacro)
@@ -2,5 +2,6 @@
 <robot xmlns:xacro="http://wiki.ros.org/xacro">
   <xacro:macro name="linear_axis" params="prefix">
-    <!-- link list -->
+    <!-- LINEAR AXIS -->
+    <!-- linear axis link list -->
     <link name="${prefix}axis">
       <inertial>
@@ -39,6 +40,5 @@
       </collision>
     </link>
-    <!-- end of link list -->
-    <!-- joint list -->
+    <!-- linear axis joint list -->
     <joint name="${prefix}cart_joint" type="prismatic">
       <parent link="${prefix}axis"/>
@@ -49,5 +49,11 @@
       <dynamics damping="0.2" friction="0" />
     </joint>
-    <!-- end of joint list -->
+    <joint name="${prefix}abb_joint" type="fixed">
+      <parent link="${prefix}cart"/>
+      <child  link="${prefix}base_link"/>
+      <origin xyz="0 0 0 " rpy="0 0 ${pi/2} "/>
+      <dynamics damping="0.2" friction="0" />
+    </joint>
+    <!-- ARE WE MISSING A WORLD TO AXIS fixed joint? for only the abb_on_axis group?-->
   </xacro:macro>
 </robot>

File: setup/catkin/princeton_cell/urdf/princeton_cell_macro.xacro (robot description, xacro)
@@ -4,6 +4,7 @@
     <!-- include files -->
     <xacro:include filename="$(find princeton_cell)/urdf/abb_on_axis_macro.xacro"/>
-    <!-- end include files -->
     <link name="world" />
+    <!-- -->
+    <!--ROBOT 2-->
     <joint name="r2_world_joint" type="fixed">
       <parent link="world" />
@@ -12,4 +13,6 @@
     </joint>
     <xacro:abb_on_axis prefix="r2_" />
+    <!-- -->
+    <!--ROBOT 1-->
     <joint name="r1_world_joint" type="fixed">
       <parent link="world" />

Commit message: swapd rpy/xyz orders (cosmetic), 0d URDF for 7600

File: setup/catkin/abb_irb4600_40_255/urdf/abb_irb4600_40_255_macro.xacro (robot description, xacro)
@@ -192,7 +192,7 @@
     <link name="${prefix}base" />
     <joint name="${prefix}base_link-base" type="fixed">
-      <origin xyz="0 0 0" rpy="0 0 0"/>
       <parent link="${prefix}base_link"/>
       <child link="${prefix}base"/>
+      <origin xyz="0 0 0" rpy="0 0 0"/>
     </joint>
   </xacro:macro>

File: setup/catkin/abb_irb4600_40_255/urdf/gripper.xacro (robot description, xacro)
@@ -21,10 +21,10 @@
       <parent link="${connected_to}"/>
       <child link="${prefix}gripper"/>
-      <origin rpy="0 0 0" xyz="0 0 0"/>
+      <origin  xyz="0 0 0" rpy="0 0 0"/>
     </joint>
     <joint name="${prefix}tcp_joint" type="fixed">
-      <origin xyz="0 0 0.352" rpy="0 0 0"/>
       <parent link="${prefix}gripper"/>
       <child link="${prefix}tcp"/>
+      <origin xyz="0 0 0.352" rpy="0 0 0"/>
     </joint>
   </xacro:macro>

File: setup/catkin/abb_irb7600_400_255/urdf/abb_irb7600_400_255.urdf (robot description, URDF)
Before this commit: robot abb_irb7600_400_255, 12 links, 11 joints
Joints:
- joint joint_2: origin xyz=0.410 0 0.780 rpy=0 0 0 -> xyz=0.0 0 0.0 rpy=0 0 0
- joint joint_3: origin xyz=0 0 1.075 rpy=0 0 0 -> xyz=0 0 0 rpy=0 0 0
- joint joint_4: origin xyz=0 0 0.165 rpy=0 0 0 -> xyz=0 0 0.0 rpy=0 0 0
- joint joint_5: origin xyz=2.012 0 0 rpy=0 0 0 -> xyz=0 0 0 rpy=0 0 0
- joint joint_6: origin xyz=0.250 0 0 rpy=0 0 0 -> xyz=0.0 0 0 rpy=0 0 0
- joint joint_balancer_piston: origin xyz=-0.380 0 0.6545 rpy=0 0 0 -> xyz=0 0 0 rpy=0 0 0

File: setup/catkin/abb_irb7600_400_255/urdf/abb_irb7600_400_255_macro.xacro (robot description, xacro)
@@ -138,54 +138,54 @@
     <!-- joint list -->
     <joint name="${prefix}joint_1" type="revolute">
-      <origin xyz="0 0 0" rpy="0 0 0"/>
       <parent link="${prefix}base_link"/>
       <child link="${prefix}link_1"/>
+      <origin xyz="0 0 0" rpy="0 0 0"/>
       <axis xyz="0 0 1"/>
       <limit lower="-${radians(180)}" upper="${radians(180)}" effort="0" velocity="${radians(100)}"/>
     </joint>
     <joint name="${prefix}joint_2" type="revolute">
-      <origin xyz="0.410 0 0.780" rpy="0 0 0"/>
       <parent link="${prefix}link_1"/>
       <child link="${prefix}link_2"/>
+      <origin xyz="0.410 0 0.780" rpy="0 0 0"/>
       <axis xyz="0 1 0"/>
       <limit lower="-${radians(60)}" upper="${radians(85)}" effort="0" velocity="${radians(60)}"/>
     </joint>
     <joint name="${prefix}joint_3" type="revolute">
-      <origin xyz="0 0 1.075" rpy="0 0 0"/>
       <parent link="${prefix}link_2"/>
       <child link="${prefix}link_3"/>
+      <origin xyz="0 0 1.075" rpy="0 0 0"/>
       <axis xyz="0 1 0"/>
       <limit lower="-${radians(180)}" upper="${radians(60)}" effort="0" velocity="${radians(60)}"/>
     </joint>
     <joint name="${prefix}joint_4" type="revolute">
-      <origin xyz="0 0 0.165" rpy="0 0 0"/>
       <parent link="${prefix}link_3"/>
       <child link="${prefix}link_4"/>
+      <origin xyz="0 0 0.165" rpy="0 0 0"/>
       <axis xyz="1 0 0"/>
       <limit lower="-${radians(300)}" upper="${radians(300)}" effort="0" velocity="${radians(100)}"/>
     </joint>
     <joint name="${prefix}joint_5" type="revolute">
-      <origin xyz="2.012 0 0" rpy="0 0 0"/>
       <parent link="${prefix}link_4"/>
       <child link="${prefix}link_5"/>
+      <origin xyz="2.012 0 0" rpy="0 0 0"/>
       <axis xyz="0 1 0"/>
       <limit lower="-${radians(100)}" upper="${radians(100)}" effort="0" velocity="${radians(100)}"/>
     </joint>
     <joint name="${prefix}joint_6" type="revolute">
-      <origin xyz="0.250 0 0" rpy="0 0 0"/>
       <parent link="${prefix}link_5"/>
       <child link="${prefix}link_6"/>
+      <origin xyz="0.250 0 0" rpy="0 0 0"/>
       <axis xyz="1 0 0"/>
       <limit lower="-${radians(360)}" upper="${radians(360)}" effort="0" velocity="${radians(190)}"/>
     </joint>
     <joint name="${prefix}joint_balancer_piston" type="fixed">
-      <origin xyz="-0.380 0 0.6545" rpy="0 0 0"/>
       <parent link="${prefix}link_1"/>
       <child link="${prefix}balancer_piston"/>
+      <origin xyz="-0.380 0 0.6545" rpy="0 0 0"/>
     </joint>
     <joint name="${prefix}joint_6-tool0" type="fixed">
-      <origin xyz="0 0 0" rpy="0 ${radians(90)} 0" />
       <parent link="${prefix}link_6" />
       <child link="${prefix}tool0" />
+      <origin xyz="0 0 0" rpy="0 ${radians(90)} 0" />
     </joint>
     <!-- -->
@@ -193,7 +193,7 @@
     <link name="${prefix}base" />
     <joint name="${prefix}base_link-base" type="fixed">
-      <origin xyz="0 0 0" rpy="0 0 0"/>
       <parent link="${prefix}base_link"/>
       <child link="${prefix}base"/>
+      <origin xyz="0 0 0" rpy="0 0 0"/>
     </joint>
   </xacro:macro>

File: setup/catkin/abb_irb7600_400_255/urdf/gripper.xacro (robot description, xacro)
@@ -21,10 +21,10 @@
       <parent link="${connected_to}"/>
       <child link="${prefix}gripper"/>
-      <origin rpy="0 0 0" xyz="0 0 0"/>
+      <origin xyz="0 0 0" rpy="0 0 0"/>
     </joint>
     <joint name="${prefix}tcp_joint" type="fixed">
-      <origin xyz="0 0 0.352" rpy="0 0 0"/>
       <parent link="${prefix}gripper"/>
       <child link="${prefix}tcp"/>
+      <origin xyz="0 0 0.352" rpy="0 0 0"/>
     </joint>
   </xacro:macro>

File: setup/catkin/princeton_cell/urdf/princeton_3rob_cell_macro.xacro (robot description, xacro)
@@ -11,5 +11,5 @@
       <parent link="world" />
       <child link = "r1_axis" />
-      <origin rpy="0.0 0.0 3.14159" xyz="3.70 3.45 0.02"/>
+      <origin xyz="3.70 3.45 0.02" rpy="0.0 0.0 3.14159" />
     </joint>
     <xacro:abb_on_axis prefix="r1_" />

File: setup/catkin/princeton_cell/urdf/princeton_cell_macro.xacro (robot description, xacro)
@@ -10,5 +10,5 @@
       <parent link="world" />
       <child link = "r1_axis" />
-      <origin rpy="0.0 0.0 3.14159" xyz="3.70 3.45 0.02"/>
+      <origin xyz="3.70 3.45 0.02" rpy="0.0 0.0 3.14159" />
     </joint>
     <xacro:abb_on_axis prefix="r1_" />

Commit message: updated all stls for 7600, fixed one for 4600

File: setup/catkin/abb_irb4600_40_255/urdf/abb_irb4600_40_255_macro.xacro (robot description, xacro)
@@ -162,5 +162,5 @@
       <parent link="${prefix}link_3"/>
       <child  link="${prefix}link_4"/>
-      <origin xyz="0.332 0 0.175" rpy="0 -0 0 "/>
+      <origin xyz="0.332 0 0.175" rpy="0 0 0 "/>
       <axis   xyz="1 0 0"/>
       <limit lower="-6.98132" upper="6.98132" effort="10000" velocity="6.2832" />
@@ -170,5 +170,5 @@
       <parent link="${prefix}link_4"/>
       <child  link="${prefix}link_5"/>
-      <origin xyz="0.939 0 0" rpy="0 -0 0 "/>
+      <origin xyz="0.939 0 0" rpy="0 0 0 "/>
       <axis   xyz="0 1 0"/>
       <limit lower="-2.18166" upper="2.0944" effort="100000" velocity="6.2832" />
@@ -178,6 +178,6 @@
       <parent link="${prefix}link_5"/>
       <child  link="${prefix}link_6"/>
-      <origin xyz="0.135 0 0" rpy="0 1.57076 0 "/>
-      <axis   xyz="0 0 1"/>
+      <origin xyz="0.135 0 0" rpy="0 0 0 "/>
+      <axis   xyz="1 0 0"/>
       <limit lower="-6.98132" upper="6.98132" effort="100000" velocity="7.854" />
       <dynamics damping="0.2" friction="0" />
@@ -186,5 +186,5 @@
       <parent link="${prefix}link_6"/>
       <child link="${prefix}tool0"/>
-      <origin xyz="0 0 0" rpy="0 0 0"/>
+      <origin xyz="0 0 0" rpy="0 ${radians(90)} 0"/>
     </joint>
     <!-- -->

File: setup/catkin/abb_irb7600_400_255/urdf/abb_irb7600_400_255_macro.xacro (robot description, xacro)
@@ -132,5 +132,5 @@
       <parent link="${prefix}link_1"/>
       <child link="${prefix}link_2"/>
-      <origin xyz="0.0 0 0.0" rpy="0 0 0"/>
+      <origin xyz="0.410 0 0.780" rpy="0 0 0"/>
       <axis xyz="0 1 0"/>
       <limit lower="-${radians(60)}" upper="${radians(85)}" effort="0" velocity="${radians(60)}"/>
@@ -139,5 +139,5 @@
       <parent link="${prefix}link_2"/>
       <child link="${prefix}link_3"/>
-      <origin xyz="0 0 0" rpy="0 0 0"/>
+      <origin xyz="0 0 1.075" rpy="0 0 0"/>
       <axis xyz="0 1 0"/>
       <limit lower="-${radians(180)}" upper="${radians(60)}" effort="0" velocity="${radians(60)}"/>
@@ -146,5 +146,5 @@
       <parent link="${prefix}link_3"/>
       <child link="${prefix}link_4"/>
-      <origin xyz="0 0 0.0" rpy="0 0 0"/>
+      <origin xyz="0.175 0 0.165" rpy="0 0 0"/>
       <axis xyz="1 0 0"/>
       <limit lower="-${radians(300)}" upper="${radians(300)}" effort="0" velocity="${radians(100)}"/>
@@ -153,5 +153,5 @@
       <parent link="${prefix}link_4"/>
       <child link="${prefix}link_5"/>
-      <origin xyz="0 0 0" rpy="0 0 0"/>
+      <origin xyz="0.882 0 0" rpy="0 0 0"/>
       <axis xyz="0 1 0"/>
       <limit lower="-${radians(100)}" upper="${radians(100)}" effort="0" velocity="${radians(100)}"/>
@@ -160,17 +160,17 @@
       <parent link="${prefix}link_5"/>
       <child link="${prefix}link_6"/>
-      <origin xyz="0 0 0" rpy="0 0 0"/>
+      <origin xyz="0.244 0 0" rpy="0 0 0"/>
       <axis xyz="1 0 0"/>
       <limit lower="-${radians(360)}" upper="${radians(360)}" effort="0" velocity="${radians(190)}"/>
+    </joint>
+    <joint name="${prefix}joint_6-tool0" type="fixed">
+      <parent link="${prefix}link_6" />
+      <child link="${prefix}tool0" />
+      <origin xyz="0 0 0" rpy="0 ${radians(90)} 0" />
     </joint>
     <joint name="${prefix}joint_balancer_piston" type="fixed">
       <parent link="${prefix}link_1"/>
       <child link="${prefix}balancer_piston"/>
-      <origin xyz="0 0 0" rpy="0 0 0"/>
-    </joint>
-    <joint name="${prefix}joint_6-tool0" type="fixed">
-      <parent link="${prefix}link_6" />
-      <child link="${prefix}tool0" />
-      <origin xyz="1.71 0 2.02" rpy="0 ${radians(90)} 0" />
+      <origin xyz="-0.378 0 0.654" rpy="0 0 0"/>
     </joint>
     <!-- -->
