Commit message: updated 4600 xacro to define joint lims in degrees

File: setup/catkin/abb_irb4600_40_255/urdf/abb_irb4600_40_255_macro.xacro (robot description, xacro)
@@ -140,5 +140,5 @@
       <origin xyz="0 0 0" rpy="0 0 0 "/>
       <axis   xyz="0 0 1"/>
-      <limit lower="-3.14159" upper="3.14159" effort="100000" velocity="2.618" />
+      <limit lower="-${radians(180)}" upper="-${radians(180)}" effort="100000" velocity="2.618" />
       <dynamics damping="0.2" friction="0" />
     </joint>
@@ -148,5 +148,5 @@
       <origin xyz="0.175 0 0.495" rpy="0 -0 0 "/>
       <axis   xyz="0 1 0"/>
-      <limit lower="-1.5708" upper="2.61799" effort="100000" velocity="2.618" />
+      <limit lower="-${radians(75)}" upper="${radians(150)}" effort="100000" velocity="2.618" />
       <dynamics damping="0.2" friction="0" />
     </joint>
@@ -156,5 +156,5 @@
       <origin xyz="0 0 1.095" rpy="0 -0 0 "/>
       <axis   xyz="0 1 0"/>
-      <limit lower="-3.14159" upper="1.309" effort="100000" velocity="2.618" />
+      <limit lower="-${radians(180)}" upper="${radians(75)}" effort="100000" velocity="2.618" />
       <dynamics damping="0.2" friction="0" />
     </joint>
@@ -164,5 +164,5 @@
       <origin xyz="0.332 0 0.175" rpy="0 0 0 "/>
       <axis   xyz="1 0 0"/>
-      <limit lower="-6.98132" upper="6.98132" effort="10000" velocity="6.2832" />
+      <limit lower="-${radians(400)}" upper="${radians(400)}" effort="10000" velocity="6.2832" />
       <dynamics damping="0.2" friction="0" />
     </joint>
@@ -172,5 +172,5 @@
       <origin xyz="0.939 0 0" rpy="0 0 0 "/>
       <axis   xyz="0 1 0"/>
-      <limit lower="-2.18166" upper="2.0944" effort="100000" velocity="6.2832" />
+      <limit lower="-${radians(125)}" upper="${radians(120)}" effort="100000" velocity="6.2832" />
       <dynamics damping="0.2" friction="0" />
     </joint>
@@ -180,5 +180,5 @@
       <origin xyz="0.135 0 0" rpy="0 0 0 "/>
       <axis   xyz="1 0 0"/>
-      <limit lower="-6.98132" upper="6.98132" effort="100000" velocity="7.854" />
+      <limit lower="-${radians(400)}" upper="${radians(400)}" effort="100000" velocity="7.854" />
       <dynamics damping="0.2" friction="0" />
     </joint>

Commit message: added the rotated 4600 link_4 to collision folder

File: setup/catkin/abb_irb4600_40_255/urdf/abb_irb4600_40_255_macro.xacro (robot description, xacro)
@@ -146,5 +146,5 @@
       <parent link="${prefix}link_1"/>
       <child  link="${prefix}link_2"/>
-      <origin xyz="0.175 0 0.495" rpy="0 -0 0 "/>
+      <origin xyz="0.175 0 0.495" rpy="0 0 0 "/>
       <axis   xyz="0 1 0"/>
       <limit lower="-${radians(75)}" upper="${radians(150)}" effort="100000" velocity="2.618" />
@@ -154,5 +154,5 @@
       <parent link="${prefix}link_2"/>
       <child  link="${prefix}link_3"/>
-      <origin xyz="0 0 1.095" rpy="0 -0 0 "/>
+      <origin xyz="0 0 1.095" rpy="0 0 0 "/>
       <axis   xyz="0 1 0"/>
       <limit lower="-${radians(180)}" upper="${radians(75)}" effort="100000" velocity="2.618" />

Commit message: clean up all folders, delet old files, color xacro

File: setup/catkin/abb_irb4600_40_255/urdf/abb_irb4600_40_255_macro.xacro (robot description, xacro)
@@ -17,5 +17,5 @@
           <mesh filename="package://abb_irb4600_40_255/meshes/visual/base_link.stl"/>
         </geometry>
-        <xacro:material_abb_white/>
+        <xacro:material_abb_gray_white/>
       </visual>
       <collision>
@@ -23,5 +23,5 @@
           <mesh filename="package://abb_irb4600_40_255/meshes/collision/base_link.stl"/>
         </geometry>
-        <xacro:material_abb_white/>
+        <xacro:material_abb_gray_white/>
       </collision>
     </link>
@@ -36,5 +36,5 @@
           <mesh filename="package://abb_irb4600_40_255/meshes/visual/link_1.stl"/>
         </geometry>
-        <xacro:material_abb_graphite_white />
+        <xacro:material_abb_gray_white />
       </visual>
       <collision>
@@ -42,4 +42,5 @@
           <mesh filename="package://abb_irb4600_40_255/meshes/collision/link_1.stl"/>
         </geometry>
+        <xacro:material_abb_gray_white/>
       </collision>
     </link>
@@ -54,5 +55,5 @@
           <mesh filename="package://abb_irb4600_40_255/meshes/visual/link_2.stl"/>
         </geometry>
-        <xacro:material_abb_graphite_white />
+        <xacro:material_abb_gray_white/>
       </visual>
       <collision>
@@ -60,4 +61,5 @@
           <mesh filename="package://abb_irb4600_40_255/meshes/collision/link_2.stl"/>
         </geometry>
+        <xacro:material_abb_gray_white/>
       </collision>
     </link>
@@ -72,5 +74,5 @@
           <mesh filename="package://abb_irb4600_40_255/meshes/visual/link_3.stl"/>
         </geometry>
-        <xacro:material_abb_graphite_white />
+        <xacro:material_abb_gray_white/>
       </visual>
       <collision>
@@ -78,4 +80,5 @@
           <mesh filename="package://abb_irb4600_40_255/meshes/collision/link_3.stl"/>
         </geometry>
+        <xacro:material_abb_gray_white/>
       </collision>
     </link>
@@ -90,5 +93,5 @@
           <mesh filename="package://abb_irb4600_40_255/meshes/visual/link_4.stl"/>
         </geometry>
-        <xacro:material_abb_graphite_white />
+        <xacro:material_abb_gray_white/>
       </visual>
       <collision>
@@ -96,4 +99,5 @@
           <mesh filename="package://abb_irb4600_40_255/meshes/collision/link_4.stl"/>
         </geometry>
+        <xacro:material_abb_gray_white/>
       </collision>
     </link>
@@ -108,5 +112,5 @@
           <mesh filename="package://abb_irb4600_40_255/meshes/visual/link_5.stl"/>
         </geometry>
-        <xacro:material_abb_graphite_white />
+        <xacro:material_abb_gray_white/>
       </visual>
       <collision>
@@ -114,4 +118,5 @@
           <mesh filename="package://abb_irb4600_40_255/meshes/collision/link_5.stl"/>
         </geometry>
+        <xacro:material_abb_gray_white/>
       </collision>
     </link>
@@ -126,5 +131,5 @@
           <mesh filename="package://abb_irb4600_40_255/meshes/visual/link_6.stl"/>
         </geometry>
-        <xacro:material_abb_graphite_white />
+        <xacro:material_abb_gray_white/>
       </visual>
       <collision>
@@ -132,4 +137,5 @@
           <mesh filename="package://abb_irb4600_40_255/meshes/collision/link_6.stl"/>
         </geometry>
+        <xacro:material_abb_gray_white/>
       </collision>
     </link>

File: setup/catkin/abb_irb4600_40_255/urdf/gripper.xacro (robot description, xacro)
@@ -9,5 +9,5 @@
           <mesh filename="package://abb_irb4600_40_255/meshes/visual/gripper.stl"/>
         </geometry>
-        <xacro:material_abb_yellow />
+        <xacro:material_light_pink />
       </visual>
       <collision>
@@ -15,5 +15,5 @@
           <mesh filename="package://abb_irb4600_40_255/meshes/collision/gripper.stl"/>
         </geometry>
-        <xacro:material_abb_yellow />
+        <xacro:material_light_pink />
       </collision>
     </link>

File: setup/catkin/abb_irb7600_400_255/urdf/abb_irb7600_400_255_macro.xacro (robot description, xacro)
@@ -12,5 +12,5 @@
           <mesh filename="package://abb_irb7600_400_255/meshes/visual/base_link.stl"/>
         </geometry>
-        <xacro:material_abb_orange />
+        <xacro:material_abb_gray_white/>
       </visual>
       <collision>
@@ -18,5 +18,5 @@
           <mesh filename="package://abb_irb7600_400_255/meshes/collision/base_link.stl"/>
         </geometry>
-        <xacro:material_abb_orange />
+        <xacro:material_abb_gray_white/>
       </collision>
     </link>
@@ -26,5 +26,5 @@
           <mesh filename="package://abb_irb7600_400_255/meshes/visual/link_1.stl"/>
         </geometry>
-        <xacro:material_abb_orange />
+        <xacro:material_abb_gray_white/>
       </visual>
       <collision>
@@ -32,5 +32,5 @@
           <mesh filename="package://abb_irb7600_400_255/meshes/collision/link_1.stl"/>
         </geometry>
-        <xacro:material_abb_yellow />
+        <xacro:material_abb_gray_white/>
       </collision>
     </link>
@@ -40,5 +40,5 @@
           <mesh filename="package://abb_irb7600_400_255/meshes/visual/link_2.stl"/>
         </geometry>
-        <xacro:material_abb_orange />
+        <xacro:material_abb_gray_white/>
       </visual>
       <collision>
@@ -46,5 +46,5 @@
           <mesh filename="package://abb_irb7600_400_255/meshes/collision/link_2.stl"/>
         </geometry>
-        <xacro:material_abb_yellow />
+        <xacro:material_abb_gray_white/>
       </collision>
     </link>
@@ -54,5 +54,5 @@
           <mesh filename="package://abb_irb7600_400_255/meshes/visual/link_3.stl"/>
         </geometry>
-        <xacro:material_abb_orange />
+        <xacro:material_abb_gray_white/>
       </visual>
       <collision>
@@ -60,5 +60,5 @@
           <mesh filename="package://abb_irb7600_400_255/meshes/collision/link_3.stl"/>
         </geometry>
-        <xacro:material_abb_yellow />
+        <xacro:material_abb_gray_white/>
       </collision>
     </link>
@@ -68,5 +68,5 @@
           <mesh filename="package://abb_irb7600_400_255/meshes/visual/link_4.stl"/>
         </geometry>
-        <xacro:material_abb_orange />
+        <xacro:material_abb_gray_white/>
       </visual>
     <collision>
@@ -74,5 +74,5 @@
           <mesh filename="package://abb_irb7600_400_255/meshes/collision/link_4.stl"/>
         </geometry>
-        <xacro:material_abb_yellow />
+        <xacro:material_abb_gray_white/>
       </collision>
     </link>
@@ -82,5 +82,5 @@
           <mesh filename="package://abb_irb7600_400_255/meshes/visual/link_5.stl"/>
         </geometry>
-        <xacro:material_abb_orange />
+        <xacro:material_abb_gray_white/>
       </visual>
       <collision>
@@ -88,5 +88,5 @@
           <mesh filename="package://abb_irb7600_400_255/meshes/collision/link_5.stl"/>
         </geometry>
-        <xacro:material_abb_yellow />
+        <xacro:material_abb_gray_white/>
       </collision>
     </link>
@@ -96,5 +96,5 @@
           <mesh filename="package://abb_irb7600_400_255/meshes/visual/link_6.stl"/>
         </geometry>
-        <xacro:material_abb_orange />
+        <xacro:material_abb_gray_white/>
       </visual>
       <collision>
@@ -102,5 +102,5 @@
           <mesh filename="package://abb_irb7600_400_255/meshes/collision/link_6.stl"/>
         </geometry>
-        <xacro:material_abb_yellow />
+        <xacro:material_abb_gray_white/>
       </collision>
     </link>
@@ -110,5 +110,5 @@
           <mesh filename="package://abb_irb7600_400_255/meshes/visual/balancer_piston.stl"/>
         </geometry>
-        <xacro:material_abb_orange />
+        <xacro:material_abb_gray_white/>
       </visual>
       <collision>
@@ -116,5 +116,5 @@
           <mesh filename="package://abb_irb7600_400_255/meshes/collision/balancer_piston.stl"/>
         </geometry>
-        <xacro:material_abb_yellow />
+        <xacro:material_abb_gray_white/>
       </collision>
     </link>

File: setup/catkin/abb_irb7600_400_255/urdf/gripper.xacro (robot description, xacro)
@@ -10,10 +10,10 @@
         </geometry>
       </visual>
-      <xacro:material_abb_yellow />
+      <xacro:material_light_pink />
       <collision>
         <geometry>
           <mesh filename="package://abb_irb7600_400_255/meshes/collision/gripper.stl"/>
         </geometry>
-        <xacro:material_abb_yellow />
+        <xacro:material_light_pink />
       </collision>
     </link>

File: setup/catkin/abb_on_axis/urdf/linear_axis.xacro (robot description, xacro)
@@ -14,5 +14,5 @@
           <mesh filename="package://abb_on_axis/meshes/visual/axis.stl"/>
         </geometry>
-        <xacro:material_abb_white />
+        <xacro:material_abb_pebble_gray />
       </visual>
       <collision>
@@ -20,4 +20,5 @@
           <mesh filename="package://abb_on_axis/meshes/collision/axis.stl"/>
         </geometry>
+        <xacro:material_abb_pebble_gray />
       </collision>
     </link>
@@ -32,5 +33,5 @@
           <mesh filename="package://abb_on_axis/meshes/visual/cart.stl"/>
         </geometry>
-        <xacro:material_abb_white />
+        <xacro:material_abb_gray_white />
       </visual>
       <collision>
@@ -38,4 +39,5 @@
           <mesh filename="package://abb_on_axis/meshes/collision/cart.stl"/>
         </geometry>
+        <xacro:material_abb_gray_white />
       </collision>
     </link>

File: setup/catkin/abb_resources/urdf/common_colours.xacro (robot description, xacro)
@@ -36,3 +36,5 @@
   <!-- yellow, collision model -->
   <xacro:property name="colour_abb_yellow" value="1 1 0 1" />
+  <!-- light pink -->
+  <xacro:property name="colour_light_pink" value="${ 255/255} ${204/255} ${203/255} 1" />
 </robot>

File: setup/catkin/abb_resources/urdf/common_materials.xacro (robot description, xacro)
@@ -77,3 +77,8 @@
     </material>
   </xacro:macro>
+  <xacro:macro name="material_light_pink">
+    <material name="">
+      <color rgba="${colour_light_pink}"/>
+    </material>
+  </xacro:macro>
 </robot>
