Commit message: update 7600 xacro color for gripper

File: setup/catkin/abb_irb7600_400_255/urdf/gripper.xacro (robot description, xacro)
@@ -9,6 +9,6 @@
           <mesh filename="package://abb_irb7600_400_255/meshes/visual/gripper.stl"/>
         </geometry>
+        <xacro:material_light_pink />
       </visual>
-      <xacro:material_light_pink />
       <collision>
         <geometry>

File: setup/catkin/abb_resources/urdf/common_colours.xacro (robot description, xacro)
@@ -37,4 +37,4 @@
   <xacro:property name="colour_abb_yellow" value="1 1 0 1" />
   <!-- light pink -->
-  <xacro:property name="colour_light_pink" value="${ 255/255} ${204/255} ${203/255} 1" />
+  <xacro:property name="colour_light_pink" value="${255/255} ${204/255} ${203/255} 1" />
 </robot>
