Commit message: made 3rob xacro file

File: setup/catkin/abb_irb7600_400_255/urdf/abb_irb7600_400_255_macro.xacro (robot description, xacro)
@@ -3,5 +3,8 @@
   <xacro:include filename="$(find abb_resources)/urdf/common_materials.xacro"/>
   <xacro:macro name="abb_irb7600_400_255" params="prefix">
-    <!-- link list -->
+    <xacro:include filename="$(find princeton_cell)/urdf/gripper.xacro" />
+    <xacro:gripper prefix="${prefix}" connected_to="${prefix}tool0"/>
+    <!-- IRB7600-->
+    <!-- irb7600 link list -->
     <link name="${prefix}base_link">
       <visual>
@@ -131,4 +134,5 @@
       </collision>
     </link>
+    <link name="${prefix}tool0" />
     <!-- end of link list -->
     <!-- joint list -->
@@ -180,5 +184,10 @@
       <child link="${prefix}balancer_piston"/>
     </joint>
-    <!-- end of joint list -->
+    <joint name="${prefix}joint_6-tool0" type="fixed">
+      <origin xyz="0 0 0" rpy="0 ${radians(90)} 0" />
+      <parent link="${prefix}link_6" />
+      <child link="${prefix}tool0" />
+    </joint>
+    <!-- -->
     <!-- ROS-Industrial 'base' frame: base_link to ABB World Coordinates transform -->
     <link name="${prefix}base" />
@@ -188,18 +197,4 @@
       <child link="${prefix}base"/>
     </joint>
-    <!-- ROS-Industrial 'flange' frame: attachment point for EEF models -->
-    <link name="${prefix}flange"/>
-    <joint type="fixed" name="${prefix}joint_6-flange">
-      <origin xyz="0 0 0" rpy="0 0 0"/>
-      <parent link="${prefix}link_6"/>
-      <child link="${prefix}flange"/>
-    </joint>
-    <!-- ROS-Industrial 'tool0' frame: all-zeros tool frame -->
-    <link name="${prefix}tool0" />
-    <joint name="${prefix}link_6-tool0" type="fixed">
-      <origin xyz="0 0 0" rpy="0 ${radians(90)} 0" />
-      <parent link="${prefix}flange" />
-      <child link="${prefix}tool0" />
-    </joint>
   </xacro:macro>
 </robot>

File: setup/catkin/princeton_cell/urdf/princeton_3rob_cell_macro.xacro (robot description, xacro)
@@ -1,6 +1,7 @@
 <?xml version="1.0"?>
 <robot xmlns:xacro="http://wiki.ros.org/xacro">
-  <xacro:macro name="princeton_cell">
+  <xacro:macro name="princeton_3rob_cell">
     <!-- include files -->
+    <xacro:include filename="$(find abb_irb7600_400_255)/urdf/abb_irb7600_400_255_macro.xacro"/>
     <xacro:include filename="$(find princeton_cell)/urdf/abb_on_axis_macro.xacro"/>
     <link name="world" />
@@ -21,4 +22,12 @@
     </joint>
     <xacro:abb_on_axis prefix="r2_" />
+    <!-- -->
+    <!--ROBOT 3-->
+    <joint name="r3_world_joint" type="fixed">
+      <parent link="world" />
+      <child link = "r3_base_link" />
+      <origin xyz="0.0 0.0 0.0" rpy="0.0 0.0 0.0" />
+    </joint>
+    <xacro:abb_irb7600_400_255 prefix="r3_" />
   </xacro:macro>
 </robot>

Commit message: rmv visual orign fr 7600, inertial orign fr track

File: setup/catkin/abb_irb7600_400_255/urdf/abb_irb7600_400_255_macro.xacro (robot description, xacro)
@@ -9,5 +9,4 @@
     <link name="${prefix}base_link">
       <visual>
-        <origin xyz="0 0 0" rpy="0 0 0"/>
         <geometry>
           <mesh filename="package://abb_irb7600_400_255/meshes/visual/base_link.stl"/>
@@ -24,5 +23,4 @@
     <link name="${prefix}link_1">
       <visual>
-        <origin xyz="0 0 0" rpy="0 0 0"/>
         <geometry>
           <mesh filename="package://abb_irb7600_400_255/meshes/visual/link_1.stl"/>
@@ -31,5 +29,4 @@
       </visual>
       <collision>
-        <origin xyz="0 0 0" rpy="0 0 0"/>
         <geometry>
           <mesh filename="package://abb_irb7600_400_255/meshes/collision/link_1.stl"/>
@@ -40,5 +37,4 @@
     <link name="${prefix}link_2">
       <visual>
-        <origin xyz="0 0 0" rpy="0 0 0"/>
         <geometry>
           <mesh filename="package://abb_irb7600_400_255/meshes/visual/link_2.stl"/>
@@ -47,5 +43,4 @@
       </visual>
       <collision>
-        <origin xyz="0 0 0" rpy="0 0 0"/>
         <geometry>
           <mesh filename="package://abb_irb7600_400_255/meshes/collision/link_2.stl"/>
@@ -56,5 +51,4 @@
     <link name="${prefix}link_3">
       <visual>
-        <origin xyz="0 0 0" rpy="0 0 0"/>
         <geometry>
           <mesh filename="package://abb_irb7600_400_255/meshes/visual/link_3.stl"/>
@@ -63,5 +57,4 @@
       </visual>
       <collision>
-        <origin xyz="0 0 0" rpy="0 0 0"/>
         <geometry>
           <mesh filename="package://abb_irb7600_400_255/meshes/collision/link_3.stl"/>
@@ -72,5 +65,4 @@
     <link name="${prefix}link_4">
       <visual>
-        <origin xyz="2.012 0 0" rpy="0 0 0"/>
         <geometry>
           <mesh filename="package://abb_irb7600_400_255/meshes/visual/link_4.stl"/>
@@ -79,5 +71,4 @@
       </visual>
     <collision>
-        <origin xyz="2.012 0 0" rpy="0 0 0"/>
         <geometry>
           <mesh filename="package://abb_irb7600_400_255/meshes/collision/link_4.stl"/>
@@ -88,5 +79,4 @@
     <link name="${prefix}link_5">
       <visual>
-        <origin xyz="0 0 0" rpy="0 0 0"/>
         <geometry>
           <mesh filename="package://abb_irb7600_400_255/meshes/visual/link_5.stl"/>
@@ -95,5 +85,4 @@
       </visual>
       <collision>
-        <origin xyz="0 0 0" rpy="0 0 0"/>
         <geometry>
           <mesh filename="package://abb_irb7600_400_255/meshes/collision/link_5.stl"/>
@@ -104,5 +93,4 @@
     <link name="${prefix}link_6">
       <visual>
-        <origin xyz="0 0 0" rpy="0 0 0"/>
         <geometry>
           <mesh filename="package://abb_irb7600_400_255/meshes/visual/link_6.stl"/>
@@ -111,5 +99,4 @@
       </visual>
       <collision>
-        <origin xyz="0 0 0" rpy="0 0 0"/>
         <geometry>
           <mesh filename="package://abb_irb7600_400_255/meshes/collision/link_6.stl"/>
@@ -120,5 +107,4 @@
     <link name="${prefix}balancer_piston">
       <visual>
-        <origin xyz="0 0 0" rpy="0 0 0"/>
         <geometry>
           <mesh filename="package://abb_irb7600_400_255/meshes/visual/balancer_piston.stl"/>
@@ -127,5 +113,4 @@
       </visual>
       <collision>
-        <origin xyz="0 0 0" rpy="0 0 0"/>
         <geometry>
           <mesh filename="package://abb_irb7600_400_255/meshes/collision/balancer_piston.stl"/>

File: setup/catkin/princeton_cell/urdf/linear_axis.xacro (robot description, xacro)
@@ -6,5 +6,4 @@
     <link name="${prefix}axis">
       <inertial>
-        <origin xyz="0.0 0.0 0.0"/>
         <mass value="120"/>
         <inertia ixx="-4.98000" iyy="-5.95200" izz="0.82800" ixy="-0.00000" ixz="2.70000" iyz="-0.00000"/>
@@ -24,5 +23,4 @@
     <link name="${prefix}cart">
       <inertial>
-        <origin xyz="0.0 0.0 0.0"/>
         <mass value="120.00000"/>
         <inertia ixx="-4.98000" iyy="-5.95200" izz="0.82800" ixy="-0.00000" ixz="2.70000" iyz="-0.00000"/>

Commit message: updates with new robot3 gripper

File: setup/catkin/abb_irb7600_400_255/urdf/abb_irb7600_400_255_macro.xacro (robot description, xacro)
@@ -160,5 +160,5 @@
       <parent link="${prefix}link_5"/>
       <child link="${prefix}link_6"/>
-      <origin xyz="0.2435 0 0" rpy="0 0 0"/>
+      <origin xyz="0.2490 0 0" rpy="0 0 0"/>
       <axis xyz="1 0 0"/>
       <limit lower="-${radians(360)}" upper="${radians(360)}" effort="0" velocity="${radians(190)}"/>
