Commit message: fixed mesh paths for irb7600 link4

File: setup/catkin/abb_irb7600_400_255/urdf/abb_irb7600_400_255.urdf (robot description, URDF)
Before this commit: robot abb_irb7600_400_255, 12 links, 11 joints
Links:
- link link_4: geometry collision mesh filename=package://abb_irb7600_400_255/meshes/collision/link_4.stl; visual mesh filename=package://abb_irb7600_400_255/meshes/visual/link_4.stl

File: setup/catkin/abb_irb7600_400_255/urdf/abb_irb7600_400_255_macro.xacro (robot description, xacro)
@@ -74,5 +74,5 @@
         <origin xyz="2.012 0 0" rpy="0 0 0"/>
         <geometry>
-          <mesh filename="package://abb_irb7600_support/meshes/irb7600_150_350/visual/link_4.stl"/>
+          <mesh filename="package://abb_irb7600_400_255/meshes/visual/link_4.stl"/>
         </geometry>
         <xacro:material_abb_orange />
@@ -81,5 +81,5 @@
         <origin xyz="2.012 0 0" rpy="0 0 0"/>
         <geometry>
-          <mesh filename="package://abb_irb7600_support/meshes/irb7600_150_350/collision/link_4.stl"/>
+          <mesh filename="package://abb_irb7600_400_255/meshes/collision/link_4.stl"/>
         </geometry>
         <xacro:material_abb_yellow />

File: setup/catkin/princeton_cell/urdf/princeton_3rob_cell.urdf (robot description, URDF)
Before this commit: robot princeton_3rob_cell, 39 links, 38 joints
Links:
- link r3_link_4: geometry collision mesh filename=package://abb_irb7600_400_255/meshes/collision/link_4.stl; visual mesh filename=package://abb_irb7600_400_255/meshes/visual/link_4.stl

Commit message: regen all urdfs, updated 7600 xacro with 0 origins

File: setup/catkin/abb_irb7600_400_255/urdf/abb_irb7600_400_255.urdf (robot description, URDF)
Before this commit: robot abb_irb7600_400_255, 12 links, 11 joints
Joints:
- joint joint_6: origin xyz=0.0 0 0 rpy=0 0 0 -> xyz=0 0 0 rpy=0 0 0
- joint joint_6-tool0: origin xyz=0 0 0 rpy=0 1.5707963267948966 0 -> xyz=1.71 0 2.02 rpy=0 1.5707963267948966 0

File: setup/catkin/abb_irb7600_400_255/urdf/abb_irb7600_400_255_macro.xacro (robot description, xacro)
@@ -132,5 +132,5 @@
       <parent link="${prefix}link_1"/>
       <child link="${prefix}link_2"/>
-      <origin xyz="0.410 0 0.780" rpy="0 0 0"/>
+      <origin xyz="0.0 0 0.0" rpy="0 0 0"/>
       <axis xyz="0 1 0"/>
       <limit lower="-${radians(60)}" upper="${radians(85)}" effort="0" velocity="${radians(60)}"/>
@@ -139,5 +139,5 @@
       <parent link="${prefix}link_2"/>
       <child link="${prefix}link_3"/>
-      <origin xyz="0 0 1.075" rpy="0 0 0"/>
+      <origin xyz="0 0 0" rpy="0 0 0"/>
       <axis xyz="0 1 0"/>
       <limit lower="-${radians(180)}" upper="${radians(60)}" effort="0" velocity="${radians(60)}"/>
@@ -146,5 +146,5 @@
       <parent link="${prefix}link_3"/>
       <child link="${prefix}link_4"/>
-      <origin xyz="0 0 0.165" rpy="0 0 0"/>
+      <origin xyz="0 0 0.0" rpy="0 0 0"/>
       <axis xyz="1 0 0"/>
       <limit lower="-${radians(300)}" upper="${radians(300)}" effort="0" velocity="${radians(100)}"/>
@@ -153,5 +153,5 @@
       <parent link="${prefix}link_4"/>
       <child link="${prefix}link_5"/>
-      <origin xyz="2.012 0 0" rpy="0 0 0"/>
+      <origin xyz="0 0 0" rpy="0 0 0"/>
       <axis xyz="0 1 0"/>
       <limit lower="-${radians(100)}" upper="${radians(100)}" effort="0" velocity="${radians(100)}"/>
@@ -160,5 +160,5 @@
       <parent link="${prefix}link_5"/>
       <child link="${prefix}link_6"/>
-      <origin xyz="0.250 0 0" rpy="0 0 0"/>
+      <origin xyz="0 0 0" rpy="0 0 0"/>
       <axis xyz="1 0 0"/>
       <limit lower="-${radians(360)}" upper="${radians(360)}" effort="0" velocity="${radians(190)}"/>
@@ -167,10 +167,10 @@
       <parent link="${prefix}link_1"/>
       <child link="${prefix}balancer_piston"/>
-      <origin xyz="-0.380 0 0.6545" rpy="0 0 0"/>
+      <origin xyz="0 0 0" rpy="0 0 0"/>
     </joint>
     <joint name="${prefix}joint_6-tool0" type="fixed">
       <parent link="${prefix}link_6" />
       <child link="${prefix}tool0" />
-      <origin xyz="0 0 0" rpy="0 ${radians(90)} 0" />
+      <origin xyz="1.71 0 2.02" rpy="0 ${radians(90)} 0" />
     </joint>
     <!-- -->

File: setup/catkin/princeton_cell/urdf/linear_axis.xacro (robot description, xacro)
@@ -6,4 +6,5 @@
     <link name="${prefix}axis">
       <inertial>
+        <origin xyz="0.0 0.0 0.0"/>
         <mass value="120"/>
         <inertia ixx="-4.98000" iyy="-5.95200" izz="0.82800" ixy="-0.00000" ixz="2.70000" iyz="-0.00000"/>
@@ -23,4 +24,5 @@
     <link name="${prefix}cart">
       <inertial>
+        <origin xyz="0.0 0.0 0.0"/>
         <mass value="120.00000"/>
         <inertia ixx="-4.98000" iyy="-5.95200" izz="0.82800" ixy="-0.00000" ixz="2.70000" iyz="-0.00000"/>

File: setup/catkin/princeton_cell/urdf/princeton_3rob_cell.urdf (robot description, URDF)
Before this commit: robot princeton_3rob_cell, 39 links, 38 joints
Joints:
- joint r3_joint_2: origin xyz=0.410 0 0.780 rpy=0 0 0 -> xyz=0.0 0 0.0 rpy=0 0 0
- joint r3_joint_3: origin xyz=0 0 1.075 rpy=0 0 0 -> xyz=0 0 0 rpy=0 0 0
- joint r3_joint_4: origin xyz=0 0 0.165 rpy=0 0 0 -> xyz=0 0 0.0 rpy=0 0 0
- joint r3_joint_5: origin xyz=2.012 0 0 rpy=0 0 0 -> xyz=0 0 0 rpy=0 0 0
- joint r3_joint_6: origin xyz=0.250 0 0 rpy=0 0 0 -> xyz=0 0 0 rpy=0 0 0
- joint r3_joint_6-tool0: origin xyz=0 0 0 rpy=0 1.5707963267948966 0 -> xyz=1.71 0 2.02 rpy=0 1.5707963267948966 0
- joint r3_joint_balancer_piston: origin xyz=-0.380 0 0.6545 rpy=0 0 0 -> xyz=0 0 0 rpy=0 0 0
- joint r3_world_joint: origin xyz=0.0 0.0 0.0 rpy=0.0 0.0 0.0 -> xyz=5.3 1.725 -0.3 rpy=0.0 0.0 3.14159

File: setup/catkin/princeton_cell/urdf/princeton_3rob_cell_macro.xacro (robot description, xacro)
@@ -27,5 +27,5 @@
       <parent link="world" />
       <child link = "r3_base_link" />
-      <origin xyz="0.0 0.0 0.0" rpy="0.0 0.0 0.0" />
+      <origin xyz="5.3 1.725 -0.3" rpy="0.0 0.0 3.14159" />
     </joint>
     <xacro:abb_irb7600_400_255 prefix="r3_" />

Commit message: updates to 7600 collision meshes

File: setup/catkin/abb_irb7600_400_255/urdf/abb_irb7600_400_255.urdf (robot description, URDF)
Before this commit: robot abb_irb7600_400_255, 12 links, 11 joints
Joints:
- joint joint_2: origin xyz=0.410 0 0.780 rpy=0 0 0 -> xyz=0.4100 0 0.8305 rpy=0 0 0
- joint joint_4: origin xyz=0.175 0 0 rpy=0 0 0 -> xyz=0.1749 0 0.1650 rpy=0 0 0
- joint joint_5: origin xyz=0.882 0 0 rpy=0 0 0 -> xyz=0.8821 0 0 rpy=0 0 0
- joint joint_6: origin xyz=0.244 0 0 rpy=0 0 0 -> xyz=0.2435 0 0 rpy=0 0 0
- joint joint_balancer_piston: origin xyz=-0.378 0 0.654 rpy=0 0 0 -> xyz=-0.3779 0 0.7044 rpy=0 0 0

File: setup/catkin/abb_irb7600_400_255/urdf/abb_irb7600_400_255_macro.xacro (robot description, xacro)
@@ -132,5 +132,5 @@
       <parent link="${prefix}link_1"/>
       <child link="${prefix}link_2"/>
-      <origin xyz="0.410 0 0.780" rpy="0 0 0"/>
+      <origin xyz="0.4100 0 0.8305" rpy="0 0 0"/>
       <axis xyz="0 1 0"/>
       <limit lower="-${radians(60)}" upper="${radians(85)}" effort="0" velocity="${radians(60)}"/>
@@ -146,5 +146,5 @@
       <parent link="${prefix}link_3"/>
       <child link="${prefix}link_4"/>
-      <origin xyz="0.175 0 0" rpy="0 0 0"/>
+      <origin xyz="0.1749 0 0.1650" rpy="0 0 0"/>
       <axis xyz="1 0 0"/>
       <limit lower="-${radians(300)}" upper="${radians(300)}" effort="0" velocity="${radians(100)}"/>
@@ -153,5 +153,5 @@
       <parent link="${prefix}link_4"/>
       <child link="${prefix}link_5"/>
-      <origin xyz="0.882 0 0" rpy="0 0 0"/>
+      <origin xyz="0.8821 0 0" rpy="0 0 0"/>
       <axis xyz="0 1 0"/>
       <limit lower="-${radians(100)}" upper="${radians(100)}" effort="0" velocity="${radians(100)}"/>
@@ -160,5 +160,5 @@
       <parent link="${prefix}link_5"/>
       <child link="${prefix}link_6"/>
-      <origin xyz="0.244 0 0" rpy="0 0 0"/>
+      <origin xyz="0.2435 0 0" rpy="0 0 0"/>
       <axis xyz="1 0 0"/>
       <limit lower="-${radians(360)}" upper="${radians(360)}" effort="0" velocity="${radians(190)}"/>
@@ -172,5 +172,5 @@
       <parent link="${prefix}link_1"/>
       <child link="${prefix}balancer_piston"/>
-      <origin xyz="-0.378 0 0.654" rpy="0 0 0"/>
+      <origin xyz="-0.3779 0 0.7044" rpy="0 0 0"/>
     </joint>
     <!-- -->

File: setup/catkin/princeton_3rob_cell/urdf/princeton_3rob_cell.urdf (robot description, URDF)
Before this commit: robot princeton_3rob_cell, 39 links, 38 joints
Joints:
- joint r3_joint_2: origin xyz=0.410 0 0.780 rpy=0 0 0 -> xyz=0.4100 0 0.8305 rpy=0 0 0
- joint r3_joint_4: origin xyz=0.175 0 0 rpy=0 0 0 -> xyz=0.1749 0 0.1650 rpy=0 0 0
- joint r3_joint_5: origin xyz=0.882 0 0 rpy=0 0 0 -> xyz=0.8821 0 0 rpy=0 0 0
- joint r3_joint_6: origin xyz=0.244 0 0 rpy=0 0 0 -> xyz=0.2435 0 0 rpy=0 0 0
- joint r3_joint_balancer_piston: origin xyz=-0.378 0 0.654 rpy=0 0 0 -> xyz=-0.3779 0 0.7044 rpy=0 0 0

Commit message: added in new gripper for 7600

File: setup/catkin/abb_irb7600_400_255/urdf/abb_irb7600_400_255.urdf (robot description, URDF)
Before this commit: robot abb_irb7600_400_255, 12 links, 11 joints
Joints:
- joint tcp_joint: origin xyz=0 0 0.352 rpy=0 0 0 -> xyz=0 0 0.1830 rpy=0 0 0

File: setup/catkin/abb_irb7600_400_255/urdf/gripper.xacro (robot description, xacro)
@@ -28,5 +28,5 @@
       <parent link="${prefix}gripper"/>
       <child link="${prefix}tcp"/>
-      <origin xyz="0 0 0.352" rpy="0 0 0"/>
+      <origin xyz="0 0 0.1830" rpy="0 0 0"/>
     </joint>
   </xacro:macro>

File: setup/catkin/princeton_3rob_cell/urdf/princeton_3rob_cell.urdf (robot description, URDF)
Before this commit: robot princeton_3rob_cell, 39 links, 38 joints
Joints:
- joint r3_tcp_joint: origin xyz=0 0 0.352 rpy=0 0 0 -> xyz=0 0 0.1830 rpy=0 0 0

Commit message: 7600 gripper to meter stl, new gripper in rh6 file

File: setup/catkin/abb_irb7600_400_255/urdf/abb_irb7600_400_255.urdf (robot description, URDF)
Before this commit: robot abb_irb7600_400_255, 12 links, 11 joints
Joints:
- joint joint_6: origin xyz=0.2435 0 0 rpy=0 0 0 -> xyz=0.2490 0 0 rpy=0 0 0
- joint tcp_joint: origin xyz=0 0 0.1830 rpy=0 0 0 -> xyz=0 0 0.2153 rpy=0 0 0

File: setup/catkin/abb_irb7600_400_255/urdf/gripper.xacro (robot description, xacro)
@@ -28,5 +28,5 @@
       <parent link="${prefix}gripper"/>
       <child link="${prefix}tcp"/>
-      <origin xyz="0 0 0.1830" rpy="0 0 0"/>
+      <origin xyz="0 0 0.2153" rpy="0 0 0"/>
     </joint>
   </xacro:macro>

File: setup/catkin/princeton_3rob_cell/urdf/princeton_3rob_cell.urdf (robot description, URDF)
Before this commit: robot princeton_3rob_cell, 39 links, 38 joints
Joints:
- joint r3_joint_6: origin xyz=0.2435 0 0 rpy=0 0 0 -> xyz=0.2490 0 0 rpy=0 0 0
- joint r3_tcp_joint: origin xyz=0 0 0.1830 rpy=0 0 0 -> xyz=0 0 0.2153 rpy=0 0 0

Commit message: fixed 7600 STL (shift base down 50.8mm)

File: setup/catkin/abb_irb7600_400_255/urdf/abb_irb7600_400_255.urdf (robot description, URDF)
Before this commit: robot abb_irb7600_400_255, 12 links, 11 joints
Joints:
- joint joint_2: origin xyz=0.4100 0 0.8305 rpy=0 0 0 -> xyz=0.4100 0 0.7797 rpy=0 0 0
- joint joint_balancer_piston: origin xyz=-0.3779 0 0.7044 rpy=0 0 0 -> xyz=-0.3779 0 0.6536 rpy=0 0 0

File: setup/catkin/abb_irb7600_400_255/urdf/abb_irb7600_400_255_macro.xacro (robot description, xacro)
@@ -132,5 +132,5 @@
       <parent link="${prefix}link_1"/>
       <child link="${prefix}link_2"/>
-      <origin xyz="0.4100 0 0.8305" rpy="0 0 0"/>
+      <origin xyz="0.4100 0 0.7797" rpy="0 0 0"/>
       <axis xyz="0 1 0"/>
       <limit lower="-${radians(60)}" upper="${radians(85)}" effort="0" velocity="${radians(60)}"/>
@@ -172,5 +172,5 @@
       <parent link="${prefix}link_1"/>
       <child link="${prefix}balancer_piston"/>
-      <origin xyz="-0.3779 0 0.7044" rpy="0 0 0"/>
+      <origin xyz="-0.3779 0 0.6536" rpy="0 0 0"/>
     </joint>
     <!-- -->

File: setup/catkin/princeton_3rob_cell/urdf/princeton_3rob_cell.urdf (robot description, URDF)
Before this commit: robot princeton_3rob_cell, 39 links, 38 joints
Links:
- link r1_gripper: geometry collision mesh filename=package://abb_irb4600_40_255/meshes/collision/gripper.stl; visual mesh filename=package://abb_irb4600_40_255/meshes/visual/gripper.stl
- link r2_gripper: geometry collision mesh filename=package://abb_irb4600_40_255/meshes/collision/gripper.stl; visual mesh filename=package://abb_irb4600_40_255/meshes/visual/gripper.stl
- link r3_gripper: geometry collision mesh filename=package://abb_irb7600_400_255/meshes/collision/gripper.stl; visual mesh filename=package://abb_irb7600_400_255/meshes/visual/gripper.stl
Joints:
- joint r3_joint_2: origin xyz=0.4100 0 0.8305 rpy=0 0 0 -> xyz=0.4100 0 0.7797 rpy=0 0 0
- joint r3_joint_balancer_piston: origin xyz=-0.3779 0 0.7044 rpy=0 0 0 -> xyz=-0.3779 0 0.6536 rpy=0 0 0

File: setup/catkin/princeton_3rob_cell/urdf/princeton_3rob_cell_normal.urdf (robot description, URDF)
Before this commit: robot princeton_3rob_cell, 39 links, 38 joints
Joints:
- joint r3_joint_2: origin xyz=0.4100 0 0.8305 rpy=0 0 0 -> xyz=0.4100 0 0.7797 rpy=0 0 0
- joint r3_joint_balancer_piston: origin xyz=-0.3779 0 0.7044 rpy=0 0 0 -> xyz=-0.3779 0 0.6536 rpy=0 0 0
