Commit message: correction to 3rob cell URDF, wobj work in 3_rob GHX

File: setup/catkin/princeton_3rob_cell/urdf/princeton_3rob_cell_OLD.urdf (robot description, URDF)
Before this commit: robot princeton_3rob_cell, 39 links, 38 joints
Links:
- link r1_gripper: geometry collision mesh filename=package://abb_irb4600_40_255/meshes/collision/gripper.stl; visual mesh filename=package://abb_irb4600_40_255/meshes/visual/gripper.stl
- link r2_gripper: geometry collision mesh filename=package://abb_irb4600_40_255/meshes/collision/gripper.stl; visual mesh filename=package://abb_irb4600_40_255/meshes/visual/gripper.stl
- link r3_gripper: geometry collision mesh filename=package://abb_irb7600_400_255/meshes/collision/gripper.stl; visual mesh filename=package://abb_irb7600_400_255/meshes/visual/gripper.stl
Joints:
- joint r1_world_joint: origin xyz=3.6986 3.4507 0.015 rpy=0.0 0.0 3.14159 -> xyz=3.70 3.45 0.02 rpy=0.0 0.0 3.14159
- joint r2_world_joint: origin xyz=0.0 0.00137 0.00036 rpy=0.0 0.0 0.0 -> xyz=0.0 0.0 0.0 rpy=0.0 0.0 0.0
- joint r3_world_joint: origin xyz=4.885 1.7193 -0.3774 rpy=0.0 0.0 3.14159 -> xyz=5.3 1.725 -0.3 rpy=0.0 0.0 3.14159
