Commit message: updated xacro offsets for 2rob and 3rob cell

File: setup/catkin/princeton_2rob_cell/urdf/princeton_2rob_cell.urdf (robot description, URDF)
Before this commit: robot princeton_2rob_cell, 27 links, 26 joints
Joints:
- joint r1_world_joint: origin xyz=3.70 3.45 0.02 rpy=0.0 0.0 3.14159 -> xyz=3.6986 3.4507 0.015 rpy=0.0 0.0 3.14159
- joint r2_world_joint: origin xyz=0.0 0.0 0.0 rpy=0.0 0.0 0.0 -> xyz=0.0 0.00137 0.00036 rpy=0.0 0.0 0.0

File: setup/catkin/princeton_2rob_cell/urdf/princeton_2rob_cell_macro.xacro (robot description, xacro)
@@ -10,5 +10,5 @@
       <parent link="world" />
       <child link = "r1_axis" />
-      <origin xyz="3.70 3.45 0.02" rpy="0.0 0.0 3.14159" />
+      <origin xyz="3.6986 3.4507 0.015" rpy="0.0 0.0 3.14159" />
     </joint>
     <xacro:abb_on_axis prefix="r1_" />
@@ -18,5 +18,5 @@
       <parent link="world" />
       <child link = "r2_axis" />
-      <origin xyz="0.0 0.0 0.0" rpy="0.0 0.0 0.0" />
+      <origin xyz="0.0 0.00137 0.00036" rpy="0.0 0.0 0.0" />
     </joint>
     <xacro:abb_on_axis prefix="r2_" />

File: setup/catkin/princeton_3rob_cell/urdf/princeton_3rob_cell.urdf (robot description, URDF)
Before this commit: robot princeton_3rob_cell, 39 links, 38 joints
Links:
- link r1_gripper: geometry collision mesh filename=package://abb_irb4600_40_255/meshes/collision/gripper.stl; visual mesh filename=package://abb_irb4600_40_255/meshes/visual/gripper.stl
- link r2_gripper: geometry collision mesh filename=package://abb_irb4600_40_255/meshes/collision/gripper.stl; visual mesh filename=package://abb_irb4600_40_255/meshes/visual/gripper.stl
- link r3_gripper: geometry collision mesh filename=package://abb_irb7600_400_255/meshes/collision/gripper.stl; visual mesh filename=package://abb_irb7600_400_255/meshes/visual/gripper.stl

File: setup/catkin/princeton_3rob_cell/urdf/princeton_3rob_cell_macro.xacro (robot description, xacro)
@@ -11,5 +11,5 @@
       <parent link="world" />
       <child link = "r1_axis" />
-      <origin rpy="0.0 0.0 3.14159" xyz="3.70 3.45 0.02"/>
+      <origin  xyz="3.6986 3.4507 0.015" rpy="0.0 0.0 3.14159"/>
     </joint>
     <xacro:abb_on_axis prefix="r1_" />
@@ -19,5 +19,5 @@
       <parent link="world" />
       <child link = "r2_axis" />
-      <origin xyz="0.0 0.0 0.0" rpy="0.0 0.0 0.0" />
+      <origin xyz="0.0 0.00137 0.00036" rpy="0.0 0.0 0.0" />
     </joint>
     <xacro:abb_on_axis prefix="r2_" />
@@ -27,5 +27,5 @@
       <parent link="world" />
       <child link = "r3_base_link" />
-      <origin xyz="5.3 1.725 -0.3" rpy="0.0 0.0 3.14159"/>
+      <origin xyz="4.885 1.7193 -0.3774" rpy="0.0 0.0 3.14159"/>
     </joint>
     <xacro:abb_irb7600_400_255 prefix="r3_" />
