Commit message: swap back to gripper URDF

File: setup/catkin/princeton_2rob_cell/urdf/princeton_2rob_cell_macro.xacro (robot description, xacro)
@@ -10,5 +10,5 @@
       <parent link="world" />
       <child link = "r1_axis" />
-      <origin xyz="3.6986 3.4507 0.015" rpy="0.0 0.0 3.14159" />
+      <origin xyz="3.6970 3.4496 0.0165" rpy="0.0 0.0 3.14159" />
     </joint>
     <xacro:abb_on_axis prefix="r1_" />
@@ -18,5 +18,5 @@
       <parent link="world" />
       <child link = "r2_axis" />
-      <origin xyz="0.0 0.00137 0.00036" rpy="0.0 0.0 0.0" />
+      <origin xyz="0.0 0.00178 0.00044" rpy="0.0 0.0 0.0" />
     </joint>
     <xacro:abb_on_axis prefix="r2_" />

File: setup/catkin/princeton_3rob_cell/urdf/princeton_3rob_cell.urdf (robot description, URDF)
Before this commit: robot princeton_3rob_cell, 39 links, 38 joints
Links:
- link r1_gripper: geometry collision mesh filename=package://abb_irb4600_40_255/meshes/collision/gripper.stl; visual mesh filename=package://abb_irb4600_40_255/meshes/visual/gripper.stl
- link r2_gripper: geometry collision mesh filename=package://abb_irb4600_40_255/meshes/collision/gripper.stl; visual mesh filename=package://abb_irb4600_40_255/meshes/visual/gripper.stl
- link r3_gripper: geometry collision mesh filename=package://abb_irb7600_400_255/meshes/collision/gripper.stl; visual mesh filename=package://abb_irb7600_400_255/meshes/visual/gripper.stl
Joints:
- joint r1_tcp_joint: origin xyz=-0.000441033 -0.0000930574 0.1642732 rpy=0 0 0 -> xyz=0 0 0.352 rpy=0 0 0
- joint r2_tcp_joint: origin xyz=0.000473456 0.000169985 0.163856 rpy=0 0 0 -> xyz=0 0 0.352 rpy=0 0 0
- joint r3_tcp_joint: origin xyz=0.000583723 0.0000236933 0.0779321 rpy=0 0 0 -> xyz=0 0 0.2153 rpy=0 0 0

File: setup/catkin/princeton_3rob_cell/urdf/princeton_3rob_cell_CALIBRATION.urdf (robot description, URDF)
Before this commit: robot princeton_3rob_cell, 39 links, 38 joints
Links:
- link r1_gripper: geometry collision mesh filename=package://abb_irb4600_40_255/meshes/collision/calibration_t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; visual mesh filename=package://abb_irb4600_40_255/meshes/visual/calibration_tool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
- link r2_gripper: geometry collision mesh filename=package://abb_irb4600_40_255/meshes/collision/calibration_t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; visual mesh filename=package://abb_irb4600_40_255/meshes/visual/calibration_tool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
- link r3_gripper: geometry collision mesh filename=package://abb_irb7600_400_255/meshes/collision/calibration_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; visual mesh filename=package://abb_irb7600_400_255/meshes/visual/calibration_too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
Joints:
- joint r1_tcp_joint: origin xyz=0 0 0.352 rpy=0 0 0 -> xyz=-0.000441033 -0.0000930574 0.1642732 rpy=0 0 0
- joint r2_tcp_joint: origin xyz=0 0 0.352 rpy=0 0 0 -> xyz=0.000473456 0.000169985 0.163856 rpy=0 0 0
- joint r2_world_joint: origin xyz=0.0 0.00178 0.00036 rpy=0.0 0.0 0.0 -> xyz=0.0 0.00178 0.00044 rpy=0.0 0.0 0.0
- joint r3_tcp_joint: origin xyz=0 0 0.2153 rpy=0 0 0 -> xyz=0.000583723 0.0000236933 0.0779321 rpy=0 0 0
- joint r3_world_joint: origin xyz=4.885 1.7193 -0.3266 rpy=0.0 0.0 3.14159 -> xyz=4.886272 1.716257 -0.322108 rpy=-0.019001374398830925 0.00022822725853081357 3.1326456328791554

File: setup/catkin/princeton_3rob_cell/urdf/princeton_3rob_cell_macro.xacro (robot description, xacro)
@@ -11,5 +11,5 @@
       <parent link="world" />
       <child link = "r1_axis" />
-      <origin  xyz="3.6986 3.4507 0.015" rpy="0.0 0.0 3.14159"/>
+      <origin  xyz="3.6970 3.4496 0.0165" rpy="0.0 0.0 3.14159"/>
     </joint>
     <xacro:abb_on_axis prefix="r1_" />
@@ -19,5 +19,5 @@
       <parent link="world" />
       <child link = "r2_axis" />
-      <origin xyz="0.0 0.00137 0.00036" rpy="0.0 0.0 0.0" />
+      <origin xyz="0.0 0.00178 0.00044" rpy="0.0 0.0 0.0" />
     </joint>
     <xacro:abb_on_axis prefix="r2_" />
@@ -27,5 +27,5 @@
       <parent link="world" />
       <child link = "r3_base_link" />
-      <origin xyz="4.885 1.7193 -0.3774" rpy="0.0 0.0 3.14159"/>
+      <origin xyz="4.886272 1.716257 -0.322108" rpy="-0.019001374398830925 0.00022822725853081357 3.1326456328791554"/>
     </joint>
     <xacro:abb_irb7600_400_255 prefix="r3_" />
