Commit message: troubleshoot URDF, added notes in readme/bashrc

File: setup/catkin/robot_on_gantry/urdf/linear_axis.xacro (robot description, xacro)
@@ -106,5 +106,5 @@
     </joint>
     <joint name="${prefix}abb_joint" type="fixed">
-      <parent link="${prefix}cart"/>
+      <parent link="${prefix}Zcart"/>
       <child  link="${prefix}base_link"/>
       <origin xyz="0 0 0 " rpy="0 0 ${pi/2} "/>
