Commit message: Start update to BAR URDF, 6620 stls

File: setup/catkin/bar_lab/urdf/bar_lab.urdf (robot description, URDF)
Before this commit: robot bar_lab, 25 links, 24 joints
Joints:
- joint bridge1_joint_EA_X: limit upper=37.206 effort=100000.0 velocity=2.618 -> lower=0.0 upper=13.005 effort=100000.0 velocity=2.618
- joint robot1_joint_EA_Y: limit upper=9.65 effort=100000.0 velocity=2.618 -> lower=0.0 upper=9.65 effort=100000.0 velocity=2.618
- joint robot1_joint_EA_Z: limit lower=0.0 upper=4.713 effort=100000.0 velocity=2.618 -> lower=2.956 upper=4.706 effort=100000.0 velocity=2.618
- joint robot2_joint_2: origin xyz=0.175 0.0 0.495 rpy=0.0 0.0 0.0 -> xyz=0.320 0.0 0.680 rpy=0.0 0.0 0.0
- joint robot2_joint_3: origin xyz=0.0 0.0 1.095 rpy=0.0 0.0 0.0 -> xyz=0.0 0.0 0.974 rpy=0.0 0.0 0.0
- joint robot2_joint_EA_Y: limit upper=9.65 effort=100000.0 velocity=2.618 -> lower=0.0 upper=9.65 effort=100000.0 velocity=2.618
- joint robot2_joint_EA_Z: limit lower=0.0 upper=4.713 effort=100000.0 velocity=2.618 -> lower=2.956 upper=4.706 effort=100000.0 velocity=2.618

Commit message: Updated BAR lab robot to IRB6620
Decent 6620 model, but requires some small fixes still. Working with 3D designer to fix.

File: setup/catkin/bar_lab/urdf/bar_lab.urdf (robot description, URDF)
Before this commit: robot bar_lab, 25 links, 24 joints
Links:
- link robot1_base_link: geometry collision mesh filename=package://abb_irb6620/meshes/collision/base_link.stl; visual mesh filename=package://abb_irb6620/meshes/visual/base_link.stl
- link robot1_link_1: geometry collision mesh filename=package://abb_irb6620/meshes/collision/link_1.stl; visual mesh filename=package://abb_irb6620/meshes/visual/link_1.stl
- link robot1_link_2: geometry collision mesh filename=package://abb_irb6620/meshes/collision/link_2.stl; visual mesh filename=package://abb_irb6620/meshes/visual/link_2.stl
- link robot1_link_3: geometry collision mesh filename=package://abb_irb6620/meshes/collision/link_3.stl; visual mesh filename=package://abb_irb6620/meshes/visual/link_3.stl
- link robot1_link_4: geometry collision mesh filename=package://abb_irb6620/meshes/collision/link_4.stl; visual mesh filename=package://abb_irb6620/meshes/visual/link_4.stl
- link robot1_link_5: geometry collision mesh filename=package://abb_irb6620/meshes/collision/link_5.stl; visual mesh filename=package://abb_irb6620/meshes/visual/link_5.stl
- link robot1_link_6: geometry collision mesh filename=package://abb_irb6620/meshes/collision/link_6.stl; visual mesh filename=package://abb_irb6620/meshes/visual/link_6.stl
- link robot2_base_link: geometry collision mesh filename=package://abb_irb6620/meshes/collision/base_link.stl; visual mesh filename=package://abb_irb6620/meshes/visual/base_link.stl
- link robot2_link_1: geometry collision mesh filename=package://abb_irb6620/meshes/collision/link_1.stl; visual mesh filename=package://abb_irb6620/meshes/visual/link_1.stl
- link robot2_link_2: geometry collision mesh filename=package://abb_irb6620/meshes/collision/link_2.stl; visual mesh filename=package://abb_irb6620/meshes/visual/link_2.stl
- link robot2_link_3: geometry collision mesh filename=package://abb_irb6620/meshes/collision/link_3.stl; visual mesh filename=package://abb_irb6620/meshes/visual/link_3.stl
- link robot2_link_4: geometry collision mesh filename=package://abb_irb6620/meshes/collision/link_4.stl; visual mesh filename=package://abb_irb6620/meshes/visual/link_4.stl
- link robot2_link_5: geometry collision mesh filename=package://abb_irb6620/meshes/collision/link_5.stl; visual mesh filename=package://abb_irb6620/meshes/visual/link_5.stl
- link robot2_link_6: geometry collision mesh filename=package://abb_irb6620/meshes/collision/link_6.stl; visual mesh filename=package://abb_irb6620/meshes/visual/link_6.stl
Joints:
- joint robot1_joint_1: limit lower=-3.14159265359 upper=3.14159265359 effort=100000.0 velocity=2.618 -> lower=-2.96706 upper=2.96706 effort=100000.0 velocity=2.618
- joint robot1_joint_2: limit lower=-1.57079632679 upper=2.61799387799 effort=100000.0 velocity=2.618 -> lower=-1.13446 upper=2.44346 effort=100000.0 velocity=2.618; origin xyz=0.175 0.0 0.495 rpy=0.0 0.0 0.0 -> xyz=0.3200 0.0 0.6800 rpy=0.0 0.0 0.0
- joint robot1_joint_3: limit lower=-3.14159265359 upper=1.308996939 effort=100000.0 velocity=2.618 -> lower=-3.14159 upper=1.22173 effort=100000.0 velocity=2.618; origin xyz=0.0 0.0 1.095 rpy=0.0 0.0 0.0 -> xyz=0.0 0.0 0.9741 rpy=0.0 0.0 0.0
- joint robot1_joint_4: limit lower=-6.98131700798 upper=6.98131700798 effort=10000.0 velocity=6.2832 -> lower=-5.23599 upper=5.23599 effort=10000.0 velocity=6.2832; origin xyz=0.331 0.0 0.175 rpy=0.0 0.0 0.0 -> xyz=0.1946 0.0 0.1988 rpy=0.0 0.0 0.0
- joint robot1_joint_5: limit lower=-2.18166 upper=2.18166156499 effort=100000.0 velocity=6.2832 -> lower=-2.26893 upper=2.26893 effort=100000.0 velocity=6.2832; origin xyz=0.939 0.0 0.0 rpy=0.0 0.0 0.0 -> xyz=0.6924 0.0 0.0 rpy=0.0 0.0 0.0
- joint robot1_joint_6: limit lower=-6.98131700798 upper=6.98131700798 effort=100000.0 velocity=7.854 -> lower=-5.23599 upper=5.23599 effort=100000.0 velocity=7.854; origin xyz=0.135 0.0 0.0 rpy=0.0 1.57079632679 0.0 -> xyz=0.174 0.0 0.0 rpy=0.0 0.0 0.0
- joint robot2_joint_1: limit lower=-3.14159265359 upper=3.14159265359 effort=100000.0 velocity=2.618 -> lower=-2.96706 upper=2.96706 effort=100000.0 velocity=2.618
- joint robot2_joint_2: limit lower=-1.57079632679 upper=2.61799387799 effort=100000.0 velocity=2.618 -> lower=-1.13446 upper=2.44346 effort=100000.0 velocity=2.618; origin xyz=0.320 0.0 0.680 rpy=0.0 0.0 0.0 -> xyz=0.3200 0.0 0.6800 rpy=0.0 0.0 0.0
- joint robot2_joint_3: limit lower=-3.14159265359 upper=1.308996939 effort=100000.0 velocity=2.618 -> lower=-3.14159 upper=1.22173 effort=100000.0 velocity=2.618; origin xyz=0.0 0.0 0.974 rpy=0.0 0.0 0.0 -> xyz=0.0 0.0 0.9741 rpy=0.0 0.0 0.0
- joint robot2_joint_4: limit lower=-6.98131700798 upper=6.98131700798 effort=10000.0 velocity=6.2832 -> lower=-5.23599 upper=5.23599 effort=10000.0 velocity=6.2832; origin xyz=0.331 0.0 0.175 rpy=0.0 0.0 0.0 -> xyz=0.1946 0.0 0.1988 rpy=0.0 0.0 0.0
- joint robot2_joint_5: limit lower=-2.18166 upper=2.18166156499 effort=100000.0 velocity=6.2832 -> lower=-2.26893 upper=2.26893 effort=100000.0 velocity=6.2832; origin xyz=0.939 0.0 0.0 rpy=0.0 0.0 0.0 -> xyz=0.6924 0.0 0.0 rpy=0.0 0.0 0.0
- joint robot2_joint_6: limit lower=-6.98131700798 upper=6.98131700798 effort=100000.0 velocity=7.854 -> lower=-5.23599 upper=5.23599 effort=100000.0 velocity=7.854; origin xyz=0.135 0.0 0.0 rpy=0.0 1.57079632679 0.0 -> xyz=0.174 0.0 0.0 rpy=0.0 0.0 0.0

Commit message: update rotation axis on joint 6

File: setup/catkin/bar_lab/urdf/bar_lab.urdf (robot description, URDF)
Before this commit: robot bar_lab, 25 links, 24 joints
Joints:
- joint robot1_joint_6: axis 0.0 0.0 1.0 -> 1.0 0.0 0.0
- joint robot2_joint_6: axis 0.0 0.0 1.0 -> 1.0 0.0 0.0

Commit message: added nicer visual meshes

File: setup/catkin/bar_lab/urdf/bar_lab.urdf (robot description, URDF)
Before this commit: robot bar_lab, 25 links, 24 joints
Links:
- link bridge2: geometry collision mesh filename=package://bar_lab/meshes/collision/y_gantry2.stl; visual mesh filename=package://bar_lab/meshes/visual/y_gantry2.stl

Commit message: updated visual and collision meshes

File: setup/catkin/bar_lab/urdf/bar_lab.urdf (robot description, URDF)
Before this commit: robot bar_lab, 25 links, 24 joints
Links:
- link bridge1: geometry collision mesh filename=package://bar_lab/meshes/collision/y_gantry1.stl; visual mesh filename=package://bar_lab/meshes/visual/y_gantry1.stl

Commit message: Update the vizualize GHX and RH files

File: setup/catkin/bar_lab/urdf/bar_lab.urdf (robot description, URDF)
Before this commit: robot bar_lab, 25 links, 24 joints
Joints:
- joint robot1_joint_6-tool0: axis 1.0 0.0 0.0 -> (none); origin xyz=0.0 0.0 0.0 rpy=0.0 0.0 0.0 -> xyz=0.0 0.0 0.0 rpy=0.0 1.5707963267948966 0.0
- joint robot2_joint_6-tool0: axis 1.0 0.0 0.0 -> (none); origin xyz=0.0 0.0 0.0 rpy=0.0 0.0 0.0 -> xyz=0.0 0.0 0.0 rpy=0.0 1.5707963267948966 0.0
